File: fpga-banks.sch (KiCad schematic (older format))
At the start: 23 parts

Commit message: Minor changes to FPGA
Parts:
- removed C?: C_10n_0402, antmicro-footprints:0402-cap, symbol antmicroCapacitors0402:C_10n_0402
- removed C?: C_1n_0402, antmicro-footprints:0402-res, symbol antmicroCapacitors0402:C_1n_0402
- removed D?: KP-1608CGCK, antmicro-footprints:LED_0603, symbol antmicroLEDIndicationDiscrete:KP-1608CGCK
- removed R?: R_100R_0402, antmicro-footprints:0402-res, symbol antmicroResistors0402:R_100R_0402
- removed R? (x2): R_140R_0402, antmicro-footprints:0402-res, symbol antmicroResistors0402:R_140R_0402
- removed R? (x3): R_1k_0402, antmicro-footprints:0402-res, symbol antmicroResistors0402:R_1k_0402
- removed U? (x2): XC7A100T-FGG484, antmicro-footprints:Xilinx_FGG484, symbol antmicroMicrocontrollers:XC7A100T-FGG484
- added J?: 62000311121, antmicro-footprints:62000311121, symbol antmicroRectangularConnectorsHeadersMalePins:62000311121
- added R? (x4): R_0R_0402, antmicro-footprints:0402-res, symbol antmicroResistors0402:R_0R_0402
Connections:
- net labels removed: V_N, V_P, XADCGND, XADCVREF, XADC_V_N, XADC_V_P
- wire segments 235 -> 232
Other:
- note added: "Configuration modes"
- note added: "This bank is unavailable on 35T"

Commit message: Added FPGA connections
Parts:
- added R? (x5): R_0R_0402, antmicro-footprints:0402-res, symbol antmicroResistors0402:R_0R_0402
Connections:
- net labels added: CHASI#, DBP_PRDY_N, DBP_PREQ_N, HPM_FW_RECOVERY, HPM_STBY_EN, HPM_STBY_RDY, HPM_STBY_RST_N, IRQ_N, PRSNT1_N, RST_PLTRST_BUF_N, RoT_CPU_RST_N, SPARE0, SPARE1, SYS_PWRBTN_N, SYS_PWROK, VCC1V35, VCC1V8
- net labels removed: QSPI_SCK, TCK, TDI_FPGA, TDO_FPGA, TMS
- wire segments 232 -> 231
- no-connect marks 0 -> 1
Other:
- note added: "Control signals from HPM"
- note removed: "TBD: should additional GPIO\npin be considered as\nBootStrap pin\n(OCP mentions 50k pulldown)"

Commit message: Updated power sequencer
Parts:
- removed R? (x5): R_0R_0402, antmicro-footprints:0402-res, symbol antmicroResistors0402:R_0R_0402
Connections:
- net labels added: VCC1V35_BANK, VCC1V8_BANK, VCC3V3_BANK
- net labels removed: VCC1V35, VCC1V8, VCCB14, VCCB15, VCCB16, VCCB34, VCCB35
- wire segments 231 -> 221
Changed lines of the file:
@@
 Wire Wire Line
 	11600 2500 12000 2500
-Text Notes 13125 725  0    118  ~ 0
-DDR3
 Text GLabel 11600 2500 0    50   BiDi ~ 0
 DDR3_DQS1-
@@
 Wire Wire Line
 	10000 8400 10000 8150
-Text GLabel 10000 8150 1    50   Input ~ 0
-VCC3V3
 $Comp
 L antmicroResistors0402:R_200R_0402 R?
@@
 Wire Wire Line
 	10800 8700 10800 8300
-Text GLabel 10800 8150 1    50   Input ~ 0
-VCC3V3
 Connection ~ 10800 8300
 Wire Wire Line
@@
 Wire Wire Line
 	9900 9750 10050 9750
-Text GLabel 10050 9750 2    50   Input ~ 0
-VCC3V3
 $Comp
 L antmicroResistors0402:R_100R_0402 R?
@@
 	1    0    0    -1
 $EndComp
-Text GLabel 9600 7550 2    50   Input ~ 0
-VCC3V3
 Wire Wire Line
 	9600 7550 9450 7550
@@
 Text GLabel 2000 1250 0    50   Input ~ 0
 VCCB13
-Text GLabel 4300 1250 2    50   Input ~ 0
-VCCB14
 Wire Wire Line
 	7600 1250 7500 1250
@@
 	7500 1250 7400 1250
 Text GLabel 6950 1250 0    50   Input ~ 0
-VCCB15
+VCC3V3_BANK
 Wire Wire Line
 	8600 1250 8700 1250
@@
 Wire Wire Line
 	9100 1250 9250 1250
-Text GLabel 9250 1250 2    50   Input ~ 0
-VCCB16
 Wire Wire Line
 	12900 1200 12800 1200
@@
 	12800 1200 12700 1200
 Text GLabel 12250 1200 0    50   Input ~ 0
-VCCB34
+VCC1V35_BANK
 Wire Wire Line
 	13900 1200 14000 1200
@@
 Wire Wire Line
 	14400 1200 14550 1200
-Text GLabel 14550 1200 2    50   Input ~ 0
-VCCB35
 Wire Notes Line
 	1350 1900 2850 1900
@@
 Text GLabel 3275 9350 0    50   Input ~ 0
 PRSNT1_N
-Text GLabel 12250 875  0    50   Input ~ 0
-VCC1V35
-Text GLabel 12675 875  2    50   Input ~ 0
-VCCB34
-Wire Wire Line
-	12325 875  12250 875
-Wire Wire Line
-	12625 875  12675 875
-$Comp
-L antmicroResistors0402:R_0R_0402 R?
-U 1 1 64C71315
-P 12475 875
-F 0 "R?" H 12475 1088 60  0000 C CNN
-F 1 "R_0R_0402" H 12475 725 60  0001 C CNN
-F 2 "antmicro-footprints:0402-res" H 12675 1075 60  0001 L CNN
-F 3 "" H 12475 875 50  0001 C CNN
-F 4 "PANASONIC" H 12675 1275 60  0001 L CNN "Manufacturer"
-F 5 "ERJ2GE0R00X" H 12675 1175 60  0001 L CNN "MPN"
-F 6 "0R" H 12475 990 50  0000 C CNN "Val"
-	1    12475 875
-	1    0    0    -1
-$EndComp
 NoConn ~ 12000 3200
 Text GLabel 11600 3300 0    50   Output ~ 0
@@
 Wire Wire Line
 	11600 3300 12000 3300
-Text GLabel 14025 875  0    50   Input ~ 0
-VCC1V35
-Text GLabel 14450 875  2    50   Input ~ 0
-VCCB35
-Wire Wire Line
-	14100 875  14025 875
-Wire Wire Line
-	14400 875  14450 875
-$Comp
-L antmicroResistors0402:R_0R_0402 R?
-U 1 1 6529BA70
-P 14250 875
-F 0 "R?" H 14250 1088 60  0000 C CNN
-F 1 "R_0R_0402" H 14250 725 60  0001 C CNN
-F 2 "antmicro-footprints:0402-res" H 14450 1075 60  0001 L CNN
-F 3 "" H 14250 875 50  0001 C CNN
-F 4 "PANASONIC" H 14450 1275 60  0001 L CNN "Manufacturer"
-F 5 "ERJ2GE0R00X" H 14450 1175 60  0001 L CNN "MPN"
-F 6 "0R" H 14250 990 50  0000 C CNN "Val"
-	1    14250 875
-	1    0    0    -1
-$EndComp
-Text GLabel 6925 900  0    50   Input ~ 0
-VCC3V3
-Text GLabel 7350 900  2    50   Input ~ 0
-VCCB15
-Wire Wire Line
-	7000 900  6925 900
-Wire Wire Line
-	7300 900  7350 900
-$Comp
-L antmicroResistors0402:R_0R_0402 R?
-U 1 1 6535C8E4
-P 7150 900
-F 0 "R?" H 7150 1113 60  0000 C CNN
-F 1 "R_0R_0402" H 7150 750 60  0001 C CNN
-F 2 "antmicro-footprints:0402-res" H 7350 1100 60  0001 L CNN
-F 3 "" H 7150 900 50  0001 C CNN
-F 4 "PANASONIC" H 7350 1300 60  0001 L CNN "Manufacturer"
-F 5 "ERJ2GE0R00X" H 7350 1200 60  0001 L CNN "MPN"
-F 6 "0R" H 7150 1015 50  0000 C CNN "Val"
-	1    7150 900
-	1    0    0    -1
-$EndComp
-Text GLabel 8725 900  0    50   Input ~ 0
-VCC3V3
-Text GLabel 9150 900  2    50   Input ~ 0
-VCCB16
-Wire Wire Line
-	8800 900  8725 900
-Wire Wire Line
-	9100 900  9150 900
-$Comp
-L antmicroResistors0402:R_0R_0402 R?
-U 1 1 655D7CE5
-P 8950 900
-F 0 "R?" H 8950 1113 60  0000 C CNN
-F 1 "R_0R_0402" H 8950 750 60  0001 C CNN
-F 2 "antmicro-footprints:0402-res" H 9150 1100 60  0001 L CNN
-F 3 "" H 8950 900 50  0001 C CNN
-F 4 "PANASONIC" H 9150 1300 60  0001 L CNN "Manufacturer"
-F 5 "ERJ2GE0R00X" H 9150 1200 60  0001 L CNN "MPN"
-F 6 "0R" H 8950 1015 50  0000 C CNN "Val"
-	1    8950 900
-	1    0    0    -1
-$EndComp
-Text GLabel 3775 975  0    50   Input ~ 0
-VCC1V8
-Text GLabel 4200 975  2    50   Input ~ 0
-VCCB14
-Wire Wire Line
-	3850 975  3775 975
-Wire Wire Line
-	4150 975  4200 975
-$Comp
-L antmicroResistors0402:R_0R_0402 R?
-U 1 1 658C9945
-P 4000 975
-F 0 "R?" H 4000 1188 60  0000 C CNN
-F 1 "R_0R_0402" H 4000 825 60  0001 C CNN
-F 2 "antmicro-footprints:0402-res" H 4200 1175 60  0001 L CNN
-F 3 "" H 4000 975 50  0001 C CNN
-F 4 "PANASONIC" H 4200 1375 60  0001 L CNN "Manufacturer"
-F 5 "ERJ2GE0R00X" H 4200 1275 60  0001 L CNN "MPN"
-F 6 "0R" H 4000 1090 50  0000 C CNN "Val"
-	1    4000 975
-	1    0    0    -1
-$EndComp
 Wire Wire Line
 	4875 2150 4550 2150
@@
 Text Notes 3300 7850 2    50   ~ 0
 Control signals from HPM
+Text Notes 13125 725  0    118  ~ 0
+DDR3
+Text GLabel 9250 1250 2    50   Input ~ 0
+VCC3V3_BANK
+Text GLabel 14550 1200 2    50   Input ~ 0
+VCC1V35_BANK
+Text GLabel 9600 7550 2    50   Input ~ 0
+VCC3V3_BANK
+Text GLabel 10000 8150 1    50   Input ~ 0
+VCC3V3_BANK
+Text GLabel 10800 8150 1    50   Input ~ 0
+VCC3V3_BANK
+Text GLabel 10050 9750 2    50   Input ~ 0
+VCC3V3_BANK
+Text GLabel 4300 1250 2    50   Input ~ 0
+VCC1V8_BANK
 $EndSCHEMATC

Commit message: Initial component placement added (to be adjusted further)
Parts:
- gave numbers to parts that had none: 14
Changed lines of the file:
@@
 SPI_ROT_MISO
 $Comp
-L antmicroMicrocontrollers:XC7A100T-FGG484 U?
+L antmicroMicrocontrollers:XC7A100T-FGG484 U1
 U 1 1 6052CB1C
 P 2550 4150
-F 0 "U?" H 3150 1175 50  0000 C CNN
+F 0 "U1" H 3150 1175 50  0000 C CNN
 F 1 "XC7A100T-FGG484" H 3150 1084 50  0000 C CNN
 F 2 "antmicro-footprints:Xilinx_FGG484" H 2250 4150 50  0001 C CNN
@@
 $EndComp
 $Comp
-L antmicroMicrocontrollers:XC7A100T-FGG484 U?
+L antmicroMicrocontrollers:XC7A100T-FGG484 U1
 U 2 1 60532D58
 P 7500 4150
-F 0 "U?" H 8100 1175 50  0000 C CNN
+F 0 "U1" H 8100 1175 50  0000 C CNN
 F 1 "XC7A100T-FGG484" H 8100 1084 50  0000 C CNN
 F 2 "antmicro-footprints:Xilinx_FGG484" H 7200 4150 50  0001 C CNN
@@
 $EndComp
 $Comp
-L antmicroMicrocontrollers:XC7A100T-FGG484 U?
+L antmicroMicrocontrollers:XC7A100T-FGG484 U1
 U 3 1 6053B1F8
 P 12800 4100
-F 0 "U?" H 13400 1125 50  0000 C CNN
+F 0 "U1" H 13400 1125 50  0000 C CNN
 F 1 "XC7A100T-FGG484" H 13400 1034 50  0000 C CNN
 F 2 "antmicro-footprints:Xilinx_FGG484" H 12500 4100 50  0001 C CNN
@@
 $EndComp
 $Comp
-L antmicroMicrocontrollers:XC7A100T-FGG484 U?
+L antmicroMicrocontrollers:XC7A100T-FGG484 U1
 U 6 1 605660E8
 P 7950 9150
-F 0 "U?" H 7921 9203 50  0000 R CNN
+F 0 "U1" H 7921 9203 50  0000 R CNN
 F 1 "XC7A100T-FGG484" H 7921 9112 50  0000 R CNN
 F 2 "antmicro-footprints:Xilinx_FGG484" H 7650 9150 50  0001 C CNN
@@
 	11100 9350 10650 9350
 $Comp
-L antmicroResistors0402:R_100R_0402 R?
+L antmicroResistors0402:R_100R_0402 R6
 U 1 1 60A2E489
 P 10000 8550
-F 0 "R?" V 9955 8620 60  0000 L CNN
+F 0 "R6" V 9955 8620 60  0000 L CNN
 F 1 "R_100R_0402" H 10000 8400 60  0001 C CNN
 F 2 "antmicro-footprints:0402-res" H 10200 8750 60  0001 L CNN
@@
 	10000 8400 10000 8150
 $Comp
-L antmicroResistors0402:R_200R_0402 R?
+L antmicroResistors0402:R_200R_0402 R8
 U 1 1 60B66864
 P 10650 8550
-F 0 "R?" V 10605 8620 60  0000 L CNN
+F 0 "R8" V 10605 8620 60  0000 L CNN
 F 1 "R_200R_0402" H 10650 8400 60  0001 C CNN
 F 2 "antmicro-footprints:0402-res" H 10850 8750 60  0001 L CNN
@@
 $EndComp
 $Comp
-L antmicroResistors0402:R_4k7_0402 R?
+L antmicroResistors0402:R_4k7_0402 R9
 U 1 1 60B67874
 P 10800 8850
-F 0 "R?" V 10755 8920 60  0000 L CNN
+F 0 "R9" V 10755 8920 60  0000 L CNN
 F 1 "R_4k7_0402" H 10800 8700 60  0001 C CNN
 F 2 "antmicro-footprints:0402-res" H 11000 9050 60  0001 L CNN
@@
 Connection ~ 10800 9550
 $Comp
-L antmicroResistors0402:R_4k7_0402 R?
+L antmicroResistors0402:R_4k7_0402 R10
 U 1 1 60BCAC0A
 P 10950 8550
-F 0 "R?" V 10905 8620 60  0000 L CNN
+F 0 "R10" V 10905 8620 60  0000 L CNN
 F 1 "R_4k7_0402" H 10950 8400 60  0001 C CNN
 F 2 "antmicro-footprints:0402-res" H 11150 8750 60  0001 L CNN
@@
 	10800 8150 10800 8300
 $Comp
-L antmicroResistors0402:R_4k7_0402 R?
+L antmicroResistors0402:R_4k7_0402 R5
 U 1 1 60C6C820
 P 9750 9750
-F 0 "R?" H 9750 9537 60  0000 C CNN
+F 0 "R5" H 9750 9537 60  0000 C CNN
 F 1 "R_4k7_0402" H 9750 9600 60  0001 C CNN
 F 2 "antmicro-footprints:0402-res" H 9950 9950 60  0001 L CNN
@@
 	9900 9750 10050 9750
 $Comp
-L antmicroResistors0402:R_100R_0402 R?
+L antmicroResistors0402:R_100R_0402 R7
 U 1 1 60D065C0
 P 10000 9000
-F 0 "R?" V 9955 9070 60  0000 L CNN
+F 0 "R7" V 9955 9070 60  0000 L CNN
 F 1 "R_100R_0402" H 10000 8850 60  0001 C CNN
 F 2 "antmicro-footprints:0402-res" H 10200 9200 60  0001 L CNN
@@
 $EndComp
 $Comp
-L power:GND #PWR?
+L power:GND #PWR06
 U 1 1 60D0D551
 P 10000 9150
-F 0 "#PWR?" H 10000 8900 50  0001 C CNN
+F 0 "#PWR06" H 10000 8900 50  0001 C CNN
 F 1 "GND" H 10005 8977 50  0000 C CNN
 F 2 "" H 10000 9150 50  0001 C CNN
@@
 $EndComp
 $Comp
-L antmicroPushbuttonSwitches:KMR2 S?
+L antmicroPushbuttonSwitches:KMR2 S1
 U 1 1 60DA2AC9
 P 10900 10100
-F 0 "S?" V 10854 10238 50  0000 L CNN
+F 0 "S1" V 10854 10238 50  0000 L CNN
 F 1 "KMR2" V 10945 10238 50  0000 L CNN
 F 2 "antmicro-footprints:SW_SPST_4.2x2.8" H 11100 10300 50  0001 L CNN
@@
 Connection ~ 10800 10250
 $Comp
-L power:GND #PWR?
+L power:GND #PWR07
 U 1 1 60E5F880
 P 10800 10450
-F 0 "#PWR?" H 10800 10200 50  0001 C CNN
+F 0 "#PWR07" H 10800 10200 50  0001 C CNN
 F 1 "GND" H 10805 10277 50  0000 C CNN
 F 2 "" H 10800 10450 50  0001 C CNN
@@
 	9450 10650 9450 10850
 $Comp
-L power:GND #PWR?
+L power:GND #PWR05
 U 1 1 60E9E149
 P 9450 10850
-F 0 "#PWR?" H 9450 10600 50  0001 C CNN
+F 0 "#PWR05" H 9450 10600 50  0001 C CNN
 F 1 "GND" H 9455 10677 50  0000 C CNN
 F 2 "" H 9450 10850 50  0001 C CNN
@@
 VCC3V3
 $Comp
-L power:GND #PWR?
+L power:GND #PWR02
 U 1 1 612D9DD9
 P 6250 10200
-F 0 "#PWR?" H 6250 9950 50  0001 C CNN
+F 0 "#PWR02" H 6250 9950 50  0001 C CNN
 F 1 "GND" V 6255 10072 50  0000 R CNN
 F 2 "" H 6250 10200 50  0001 C CNN
@@
 $EndComp
 $Comp
-L power:GND #PWR?
+L power:GND #PWR01
 U 1 1 612DAB50
 P 6250 9900
-F 0 "#PWR?" H 6250 9650 50  0001 C CNN
+F 0 "#PWR01" H 6250 9650 50  0001 C CNN
 F 1 "GND" V 6255 9772 50  0000 R CNN
 F 2 "" H 6250 9900 50  0001 C CNN
@@
 $EndComp
 $Comp
-L antmicroCapacitorsmisc:C_47u_1210 C?
+L antmicroCapacitorsmisc:C_47u_1210 C1
 U 1 1 6143B808
 P 9450 7800
-F 0 "C?" H 9565 7845 60  0000 L CNN
+F 0 "C1" H 9565 7845 60  0000 L CNN
 F 1 "C_47u_1210" H 9450 7650 60  0001 C CNN
 F 2 "antmicro-footprints:1210-cap" H 9650 8000 60  0001 L CNN
@@
 	9450 7550 9050 7550
 $Comp
-L power:GND #PWR?
+L power:GND #PWR04
 U 1 1 6148AC43
 P 9450 7950
-F 0 "#PWR?" H 9450 7700 50  0001 C CNN
+F 0 "#PWR04" H 9450 7700 50  0001 C CNN
 F 1 "GND" H 9455 7777 50  0000 C CNN
 F 2 "" H 9450 7950 50  0001 C CNN
@@
 	9450 10350 9450 10550
 $Comp
-L antmicroResistors0402:R_0R_0402 R?
+L antmicroResistors0402:R_0R_0402 R1
 U 1 1 648CDBE7
 P 6575 9775
-F 0 "R?" H 6575 9988 60  0000 C CNN
+F 0 "R1" H 6575 9988 60  0000 C CNN
 F 1 "R_0R_0402" H 6575 9625 60  0001 C CNN
 F 2 "antmicro-footprints:0402-res" H 6775 9975 60  0001 L CNN
@@
 $EndComp
 $Comp
-L antmicroResistors0402:R_0R_0402 R?
+L antmicroResistors0402:R_0R_0402 R2
 U 1 1 648CE50A
 P 6575 9900
-F 0 "R?" H 6575 10113 60  0000 C CNN
+F 0 "R2" H 6575 10113 60  0000 C CNN
 F 1 "R_0R_0402" H 6575 9750 60  0001 C CNN
 F 2 "antmicro-footprints:0402-res" H 6775 10100 60  0001 L CNN
@@
 $EndComp
 $Comp
-L antmicroResistors0402:R_0R_0402 R?
+L antmicroResistors0402:R_0R_0402 R3
 U 1 1 648D070F
 P 6575 10075
-F 0 "R?" H 6575 10288 60  0000 C CNN
+F 0 "R3" H 6575 10288 60  0000 C CNN
 F 1 "R_0R_0402" H 6575 9925 60  0001 C CNN
 F 2 "antmicro-footprints:0402-res" H 6775 10275 60  0001 L CNN
@@
 $EndComp
 $Comp
-L antmicroResistors0402:R_0R_0402 R?
+L antmicroResistors0402:R_0R_0402 R4
 U 1 1 648D0718
 P 6575 10200
-F 0 "R?" H 6575 10413 60  0000 C CNN
+F 0 "R4" H 6575 10413 60  0000 C CNN
 F 1 "R_0R_0402" H 6575 10050 60  0001 C CNN
 F 2 "antmicro-footprints:0402-res" H 6775 10400 60  0001 L CNN
@@
 	6775 10075 6725 10075
 $Comp
-L antmicroRectangularConnectorsHeadersMalePins:62000311121 J?
+L antmicroRectangularConnectorsHeadersMalePins:62000311121 J1
 U 1 1 649873F1
 P 6525 10500
-F 0 "J?" H 6583 10733 50  0000 C CNN
+F 0 "J1" H 6583 10733 50  0000 C CNN
 F 1 "62000311121" H 6575 10300 50  0001 C CNN
 F 2 "antmicro-footprints:62000311121" H 6625 10750 60  0001 L CNN
@@
 	6800 10400 6675 10400
 $Comp
-L power:GND #PWR?
+L power:GND #PWR03
 U 1 1 649B5B60
 P 6825 10600
-F 0 "#PWR?" H 6825 10350 50  0001 C CNN
+F 0 "#PWR03" H 6825 10350 50  0001 C CNN
 F 1 "GND" V 6830 10472 50  0000 R CNN
 F 2 "" H 6825 10600 50  0001 C CNN

Commit message: Minor fixes in component placement
Changed lines of the file:
@@
 Comment4 ""
 $EndDescr
-Text GLabel 6325 2350 0    50   Input ~ 0
+Text GLabel 15175 2300 2    50   Input ~ 0
 RGMII_RX_DV
-Text GLabel 6325 2050 0    50   Output ~ 0
+Text GLabel 15175 2000 2    50   Output ~ 0
 ETH_MDC
-Text GLabel 6325 3450 0    50   BiDi ~ 0
+Text GLabel 15175 3400 2    50   BiDi ~ 0
 ETH_MDIO
-Text GLabel 6325 3150 0    50   Output ~ 0
+Text GLabel 15175 3100 2    50   Output ~ 0
 RGMII_TX_DV
-Text GLabel 6325 3250 0    50   Output ~ 0
+Text GLabel 15175 3200 2    50   Output ~ 0
 RGMII_TXD0
-Text GLabel 6325 3350 0    50   Output ~ 0
+Text GLabel 15175 3300 2    50   Output ~ 0
 RGMII_TXD1
-Text GLabel 6325 3050 0    50   Output ~ 0
+Text GLabel 15175 3000 2    50   Output ~ 0
 RGMII_TXD2
-Text GLabel 6325 3550 0    50   Input ~ 0
+Text GLabel 15175 3500 2    50   Input ~ 0
 RGMII_TXD3
-Text GLabel 6325 3650 0    50   Input ~ 0
+Text GLabel 15175 3600 2    50   Input ~ 0
 RGMII_TX_CLK
-Text GLabel 6325 2450 0    50   Input ~ 0
+Text GLabel 15175 2400 2    50   Input ~ 0
 RGMII_RXD0
-Text GLabel 6325 2550 0    50   Input ~ 0
+Text GLabel 15175 2500 2    50   Input ~ 0
 RGMII_RXD1
-Text GLabel 6325 3750 0    50   Input ~ 0
+Text GLabel 15175 3700 2    50   Input ~ 0
 RGMII_RXD2
-Text GLabel 6325 2950 0    50   Input ~ 0
+Text GLabel 15175 2900 2    50   Input ~ 0
 RGMII_RXD3
-Text GLabel 6325 2150 0    50   Input ~ 0
+Text GLabel 15175 2100 2    50   Input ~ 0
 RGMII_RX_CLK
 Wire Wire Line
-	6700 2050 6325 2050
-Wire Wire Line
-	6700 2250 6325 2250
-Wire Wire Line
-	6700 2150 6325 2150
-Wire Wire Line
-	6700 2350 6325 2350
-Wire Wire Line
-	6700 2550 6325 2550
-Wire Wire Line
-	6700 2450 6325 2450
-Wire Wire Line
-	6700 2850 6325 2850
-Wire Wire Line
-	6700 2750 6325 2750
-Wire Wire Line
-	6700 2950 6325 2950
-Wire Wire Line
-	6700 3150 6325 3150
-Wire Wire Line
-	6700 3050 6325 3050
-Wire Wire Line
-	6700 3250 6325 3250
-Wire Wire Line
-	6700 3450 6325 3450
-Wire Wire Line
-	6700 3350 6325 3350
-Wire Wire Line
-	6700 3550 6325 3550
-Wire Wire Line
-	6700 3750 6325 3750
-Wire Wire Line
-	6700 3650 6325 3650
-Text GLabel 6325 2750 0    50   Input ~ 0
+	14800 2000 15175 2000
+Wire Wire Line
+	14800 2200 15175 2200
+Wire Wire Line
+	14800 2100 15175 2100
+Wire Wire Line
+	14800 2300 15175 2300
+Wire Wire Line
+	14800 2500 15175 2500
+Wire Wire Line
+	14800 2400 15175 2400
+Wire Wire Line
+	14800 2800 15175 2800
+Wire Wire Line
+	14800 2700 15175 2700
+Wire Wire Line
+	14800 2900 15175 2900
+Wire Wire Line
+	14800 3100 15175 3100
+Wire Wire Line
+	14800 3000 15175 3000
+Wire Wire Line
+	14800 3200 15175 3200
+Wire Wire Line
+	14800 3400 15175 3400
+Wire Wire Line
+	14800 3300 15175 3300
+Wire Wire Line
+	14800 3500 15175 3500
+Wire Wire Line
+	14800 3700 15175 3700
+Wire Wire Line
+	14800 3600 15175 3600
+Text GLabel 15175 2700 2    50   Input ~ 0
 ETH_INT_N
-Text GLabel 6325 2250 0    50   Input ~ 0
+Text GLabel 15175 2200 2    50   Input ~ 0
 RGMII_REF_CLK
 Wire Wire Line
-	6700 2650 6325 2650
-Text GLabel 6325 2650 0    50   Output ~ 0
+	14800 2600 15175 2600
+Text GLabel 15175 2600 2    50   Output ~ 0
 ETH_~RESET
-Text GLabel 6325 2850 0    50   Output ~ 0
+Text GLabel 15175 2800 2    50   Output ~ 0
 RGMII_TX_CLK
 Text Notes 5725 3050 1    50   ~ 0
@@
 VCC3V3_BANK
 Text GLabel 14550 1200 2    50   Input ~ 0
-VCC1V35_BANK
+VCC3V3_BANK
 Text GLabel 9600 7550 2    50   Input ~ 0
 VCC3V3_BANK
