File: fpga-banks.sch (KiCad schematic (older format))
At the start: 14 parts, among them J1 62000311121, U1 XC7A100T-FGG484

Commit message: Update after designator unification
Parts:
- renumbered C1 to C178, J1 to J13, R1 to R81, R2 to R82, R3 to R83, R4 to R84, R5 to R85, R6 to R86, R7 to R87, R8 to R88, R9 to R89, R10 to R90, U1 to U14
Changed lines of the file:
@@
 $Descr A3 16535 11693
 encoding utf-8
-Sheet 2 10
+Sheet 10 10
 Title ""
 Date ""
@@
 SPI_ROT_MISO
 $Comp
-L antmicroMicrocontrollers:XC7A100T-FGG484 U1
+L antmicroMicrocontrollers:XC7A100T-FGG484 U14
 U 1 1 6052CB1C
 P 2550 4150
-F 0 "U1" H 3150 1175 50  0000 C CNN
+F 0 "U14" H 3150 1175 50  0000 C CNN
 F 1 "XC7A100T-FGG484" H 3150 1084 50  0000 C CNN
 F 2 "antmicro-footprints:Xilinx_FGG484" H 2250 4150 50  0001 C CNN
@@
 $EndComp
 $Comp
-L antmicroMicrocontrollers:XC7A100T-FGG484 U1
+L antmicroMicrocontrollers:XC7A100T-FGG484 U14
 U 2 1 60532D58
 P 7500 4150
-F 0 "U1" H 8100 1175 50  0000 C CNN
+F 0 "U14" H 8100 1175 50  0000 C CNN
 F 1 "XC7A100T-FGG484" H 8100 1084 50  0000 C CNN
 F 2 "antmicro-footprints:Xilinx_FGG484" H 7200 4150 50  0001 C CNN
@@
 $EndComp
 $Comp
-L antmicroMicrocontrollers:XC7A100T-FGG484 U1
+L antmicroMicrocontrollers:XC7A100T-FGG484 U14
 U 3 1 6053B1F8
 P 12800 4100
-F 0 "U1" H 13400 1125 50  0000 C CNN
+F 0 "U14" H 13400 1125 50  0000 C CNN
 F 1 "XC7A100T-FGG484" H 13400 1034 50  0000 C CNN
 F 2 "antmicro-footprints:Xilinx_FGG484" H 12500 4100 50  0001 C CNN
@@
 $EndComp
 $Comp
-L antmicroMicrocontrollers:XC7A100T-FGG484 U1
+L antmicroMicrocontrollers:XC7A100T-FGG484 U14
 U 6 1 605660E8
 P 7950 9150
-F 0 "U1" H 7921 9203 50  0000 R CNN
+F 0 "U14" H 7921 9203 50  0000 R CNN
 F 1 "XC7A100T-FGG484" H 7921 9112 50  0000 R CNN
 F 2 "antmicro-footprints:Xilinx_FGG484" H 7650 9150 50  0001 C CNN
@@
 	11100 9350 10650 9350
 $Comp
-L antmicroResistors0402:R_100R_0402 R6
+L antmicroResistors0402:R_100R_0402 R86
 U 1 1 60A2E489
 P 10000 8550
-F 0 "R6" V 9955 8620 60  0000 L CNN
+F 0 "R86" V 9955 8620 60  0000 L CNN
 F 1 "R_100R_0402" H 10000 8400 60  0001 C CNN
 F 2 "antmicro-footprints:0402-res" H 10200 8750 60  0001 L CNN
@@
 	10000 8400 10000 8150
 $Comp
-L antmicroResistors0402:R_200R_0402 R8
+L antmicroResistors0402:R_200R_0402 R88
 U 1 1 60B66864
 P 10650 8550
-F 0 "R8" V 10605 8620 60  0000 L CNN
+F 0 "R88" V 10605 8620 60  0000 L CNN
 F 1 "R_200R_0402" H 10650 8400 60  0001 C CNN
 F 2 "antmicro-footprints:0402-res" H 10850 8750 60  0001 L CNN
@@
 $EndComp
 $Comp
-L antmicroResistors0402:R_4k7_0402 R9
+L antmicroResistors0402:R_4k7_0402 R89
 U 1 1 60B67874
 P 10800 8850
-F 0 "R9" V 10755 8920 60  0000 L CNN
+F 0 "R89" V 10755 8920 60  0000 L CNN
 F 1 "R_4k7_0402" H 10800 8700 60  0001 C CNN
 F 2 "antmicro-footprints:0402-res" H 11000 9050 60  0001 L CNN
@@
 Connection ~ 10800 9550
 $Comp
-L antmicroResistors0402:R_4k7_0402 R10
+L antmicroResistors0402:R_4k7_0402 R90
 U 1 1 60BCAC0A
 P 10950 8550
-F 0 "R10" V 10905 8620 60  0000 L CNN
+F 0 "R90" V 10905 8620 60  0000 L CNN
 F 1 "R_4k7_0402" H 10950 8400 60  0001 C CNN
 F 2 "antmicro-footprints:0402-res" H 11150 8750 60  0001 L CNN
@@
 	10800 8150 10800 8300
 $Comp
-L antmicroResistors0402:R_4k7_0402 R5
+L antmicroResistors0402:R_4k7_0402 R85
 U 1 1 60C6C820
 P 9750 9750
-F 0 "R5" H 9750 9537 60  0000 C CNN
+F 0 "R85" H 9750 9537 60  0000 C CNN
 F 1 "R_4k7_0402" H 9750 9600 60  0001 C CNN
 F 2 "antmicro-footprints:0402-res" H 9950 9950 60  0001 L CNN
@@
 	9900 9750 10050 9750
 $Comp
-L antmicroResistors0402:R_100R_0402 R7
+L antmicroResistors0402:R_100R_0402 R87
 U 1 1 60D065C0
 P 10000 9000
-F 0 "R7" V 9955 9070 60  0000 L CNN
+F 0 "R87" V 9955 9070 60  0000 L CNN
 F 1 "R_100R_0402" H 10000 8850 60  0001 C CNN
 F 2 "antmicro-footprints:0402-res" H 10200 9200 60  0001 L CNN
@@
 $EndComp
 $Comp
-L power:GND #PWR06
+L power:GND #PWR085
 U 1 1 60D0D551
 P 10000 9150
-F 0 "#PWR06" H 10000 8900 50  0001 C CNN
+F 0 "#PWR085" H 10000 8900 50  0001 C CNN
 F 1 "GND" H 10005 8977 50  0000 C CNN
 F 2 "" H 10000 9150 50  0001 C CNN
@@
 Connection ~ 10800 10250
 $Comp
-L power:GND #PWR07
+L power:GND #PWR086
 U 1 1 60E5F880
 P 10800 10450
-F 0 "#PWR07" H 10800 10200 50  0001 C CNN
+F 0 "#PWR086" H 10800 10200 50  0001 C CNN
 F 1 "GND" H 10805 10277 50  0000 C CNN
 F 2 "" H 10800 10450 50  0001 C CNN
@@
 	9450 10650 9450 10850
 $Comp
-L power:GND #PWR05
+L power:GND #PWR084
 U 1 1 60E9E149
 P 9450 10850
-F 0 "#PWR05" H 9450 10600 50  0001 C CNN
+F 0 "#PWR084" H 9450 10600 50  0001 C CNN
 F 1 "GND" H 9455 10677 50  0000 C CNN
 F 2 "" H 9450 10850 50  0001 C CNN
@@
 VCC3V3
 $Comp
-L power:GND #PWR02
+L power:GND #PWR081
 U 1 1 612D9DD9
 P 6250 10200
-F 0 "#PWR02" H 6250 9950 50  0001 C CNN
+F 0 "#PWR081" H 6250 9950 50  0001 C CNN
 F 1 "GND" V 6255 10072 50  0000 R CNN
 F 2 "" H 6250 10200 50  0001 C CNN
@@
 $EndComp
 $Comp
-L power:GND #PWR01
+L power:GND #PWR080
 U 1 1 612DAB50
 P 6250 9900
-F 0 "#PWR01" H 6250 9650 50  0001 C CNN
+F 0 "#PWR080" H 6250 9650 50  0001 C CNN
 F 1 "GND" V 6255 9772 50  0000 R CNN
 F 2 "" H 6250 9900 50  0001 C CNN
@@
 $EndComp
 $Comp
-L antmicroCapacitorsmisc:C_47u_1210 C1
+L antmicroCapacitorsmisc:C_47u_1210 C178
 U 1 1 6143B808
 P 9450 7800
-F 0 "C1" H 9565 7845 60  0000 L CNN
+F 0 "C178" H 9565 7845 60  0000 L CNN
 F 1 "C_47u_1210" H 9450 7650 60  0001 C CNN
 F 2 "antmicro-footprints:1210-cap" H 9650 8000 60  0001 L CNN
@@
 	9450 7550 9050 7550
 $Comp
-L power:GND #PWR04
+L power:GND #PWR083
 U 1 1 6148AC43
 P 9450 7950
-F 0 "#PWR04" H 9450 7700 50  0001 C CNN
+F 0 "#PWR083" H 9450 7700 50  0001 C CNN
 F 1 "GND" H 9455 7777 50  0000 C CNN
 F 2 "" H 9450 7950 50  0001 C CNN
@@
 	9450 10350 9450 10550
 $Comp
-L antmicroResistors0402:R_0R_0402 R1
+L antmicroResistors0402:R_0R_0402 R81
 U 1 1 648CDBE7
 P 6575 9775
-F 0 "R1" H 6575 9988 60  0000 C CNN
+F 0 "R81" H 6575 9988 60  0000 C CNN
 F 1 "R_0R_0402" H 6575 9625 60  0001 C CNN
 F 2 "antmicro-footprints:0402-res" H 6775 9975 60  0001 L CNN
@@
 $EndComp
 $Comp
-L antmicroResistors0402:R_0R_0402 R2
+L antmicroResistors0402:R_0R_0402 R82
 U 1 1 648CE50A
 P 6575 9900
-F 0 "R2" H 6575 10113 60  0000 C CNN
+F 0 "R82" H 6575 10113 60  0000 C CNN
 F 1 "R_0R_0402" H 6575 9750 60  0001 C CNN
 F 2 "antmicro-footprints:0402-res" H 6775 10100 60  0001 L CNN
@@
 $EndComp
 $Comp
-L antmicroResistors0402:R_0R_0402 R3
+L antmicroResistors0402:R_0R_0402 R83
 U 1 1 648D070F
 P 6575 10075
-F 0 "R3" H 6575 10288 60  0000 C CNN
+F 0 "R83" H 6575 10288 60  0000 C CNN
 F 1 "R_0R_0402" H 6575 9925 60  0001 C CNN
 F 2 "antmicro-footprints:0402-res" H 6775 10275 60  0001 L CNN
@@
 $EndComp
 $Comp
-L antmicroResistors0402:R_0R_0402 R4
+L antmicroResistors0402:R_0R_0402 R84
 U 1 1 648D0718
 P 6575 10200
-F 0 "R4" H 6575 10413 60  0000 C CNN
+F 0 "R84" H 6575 10413 60  0000 C CNN
 F 1 "R_0R_0402" H 6575 10050 60  0001 C CNN
 F 2 "antmicro-footprints:0402-res" H 6775 10400 60  0001 L CNN
@@
 	6775 10075 6725 10075
 $Comp
-L antmicroRectangularConnectorsHeadersMalePins:62000311121 J1
+L antmicroRectangularConnectorsHeadersMalePins:62000311121 J13
 U 1 1 649873F1
 P 6525 10500
-F 0 "J1" H 6583 10733 50  0000 C CNN
+F 0 "J13" H 6583 10733 50  0000 C CNN
 F 1 "62000311121" H 6575 10300 50  0001 C CNN
 F 2 "antmicro-footprints:62000311121" H 6625 10750 60  0001 L CNN
@@
 	6800 10400 6675 10400
 $Comp
-L power:GND #PWR03
+L power:GND #PWR082
 U 1 1 649B5B60
 P 6825 10600
-F 0 "#PWR03" H 6825 10350 50  0001 C CNN
+F 0 "#PWR082" H 6825 10350 50  0001 C CNN
 F 1 "GND" V 6830 10472 50  0000 R CNN
 F 2 "" H 6825 10600 50  0001 C CNN

Commit message: Changed PCIe connection
Connections:
- net labels added: CLK_100M_PCIE_DN, CLK_100M_PCIE_DP, PCIE_BMC_RX_DN, PCIE_BMC_RX_DP, PCIE_BMC_TX_DN, PCIE_BMC_TX_DP
Other:
- note removed: "ethernet.sch"
Changed lines of the file:
@@
 $Descr A3 16535 11693
 encoding utf-8
-Sheet 10 10
+Sheet 3 10
 Title ""
 Date ""
@@
 Text GLabel 15175 2800 2    50   Output ~ 0
 RGMII_TX_CLK
-Text Notes 5725 3050 1    50   ~ 0
-ethernet.sch
 Wire Wire Line
 	11600 2000 12000 2000
@@
 Text Notes 5650 4900 1    50   ~ 0
 QSPI from SCM \nto HPM FPGA
-Text Notes 10550 6400 1    50   ~ 0
+Text Notes 10575 6400 1    50   ~ 0
 USB1 between HPM and BMC\nUSB2 between BMC and HPM expansion
 Text GLabel 6375 5050 0    50   Input ~ 0
@@
 Text GLabel 4300 1250 2    50   Input ~ 0
 VCC1V8_BANK
+Text GLabel 6700 2050 0    50   Input ~ 0
+CLK_100M_PCIE_DP
+Text GLabel 6700 2150 0    50   Input ~ 0
+CLK_100M_PCIE_DN
+Text GLabel 6700 2250 0    50   Input ~ 0
+PCIE_BMC_TX_DP
+Text GLabel 6700 2350 0    50   Input ~ 0
+PCIE_BMC_TX_DN
+Text GLabel 6700 2550 0    50   Input ~ 0
+PCIE_BMC_RX_DN
+Text GLabel 6700 2450 0    50   Input ~ 0
+PCIE_BMC_RX_DP
 $EndSCHEMATC

Commit message: Add local component libraries
Parts:
- C178: footprint antmicro-footprints:1210-cap -> artix-dc-scm-footprints:1210-cap; symbol antmicroCapacitorsmisc:C_47u_1210 -> artix-dc-scm:C_47u_1210
- J13: footprint antmicro-footprints:62000311121 -> artix-dc-scm-footprints:62000311121; symbol antmicroRectangularConnectorsHeadersMalePins:62000311121 -> artix-dc-scm:62000311121
- R81, R82, R83, R84: footprint antmicro-footprints:0402-res -> artix-dc-scm-footprints:0402-res; symbol antmicroResistors0402:R_0R_0402 -> artix-dc-scm:R_0R_0402
- R85, R89, R90: footprint antmicro-footprints:0402-res -> artix-dc-scm-footprints:0402-res; symbol antmicroResistors0402:R_4k7_0402 -> artix-dc-scm:R_4k7_0402
- R86, R87: footprint antmicro-footprints:0402-res -> artix-dc-scm-footprints:0402-res; symbol antmicroResistors0402:R_100R_0402 -> artix-dc-scm:R_100R_0402
- R88: footprint antmicro-footprints:0402-res -> artix-dc-scm-footprints:0402-res; symbol antmicroResistors0402:R_200R_0402 -> artix-dc-scm:R_200R_0402
- S1: footprint antmicro-footprints:SW_SPST_4.2x2.8 -> artix-dc-scm-footprints:SW_SPST_4.2x2.8; symbol antmicroPushbuttonSwitches:KMR2 -> artix-dc-scm:KMR2
- U14: footprint antmicro-footprints:Xilinx_FGG484 -> artix-dc-scm-footprints:Xilinx_FGG484; symbol antmicroMicrocontrollers:XC7A100T-FGG484 -> artix-dc-scm:XC7A100T-FGG484
Changed lines of the file:
@@
 SPI_ROT_MISO
 $Comp
-L antmicroMicrocontrollers:XC7A100T-FGG484 U14
+L artix-dc-scm:XC7A100T-FGG484 U14
 U 1 1 6052CB1C
 P 2550 4150
 F 0 "U14" H 3150 1175 50  0000 C CNN
 F 1 "XC7A100T-FGG484" H 3150 1084 50  0000 C CNN
-F 2 "antmicro-footprints:Xilinx_FGG484" H 2250 4150 50  0001 C CNN
+F 2 "artix-dc-scm-footprints:Xilinx_FGG484" H 2250 4150 50  0001 C CNN
 F 3 "" H 2250 4150 50  0000 C CNN
 	1    2550 4150
@@
 $EndComp
 $Comp
-L antmicroMicrocontrollers:XC7A100T-FGG484 U14
+L artix-dc-scm:XC7A100T-FGG484 U14
 U 2 1 60532D58
 P 7500 4150
 F 0 "U14" H 8100 1175 50  0000 C CNN
 F 1 "XC7A100T-FGG484" H 8100 1084 50  0000 C CNN
-F 2 "antmicro-footprints:Xilinx_FGG484" H 7200 4150 50  0001 C CNN
+F 2 "artix-dc-scm-footprints:Xilinx_FGG484" H 7200 4150 50  0001 C CNN
 F 3 "" H 7200 4150 50  0000 C CNN
 	2    7500 4150
@@
 $EndComp
 $Comp
-L antmicroMicrocontrollers:XC7A100T-FGG484 U14
+L artix-dc-scm:XC7A100T-FGG484 U14
 U 3 1 6053B1F8
 P 12800 4100
 F 0 "U14" H 13400 1125 50  0000 C CNN
 F 1 "XC7A100T-FGG484" H 13400 1034 50  0000 C CNN
-F 2 "antmicro-footprints:Xilinx_FGG484" H 12500 4100 50  0001 C CNN
+F 2 "artix-dc-scm-footprints:Xilinx_FGG484" H 12500 4100 50  0001 C CNN
 F 3 "" H 12500 4100 50  0000 C CNN
 	3    12800 4100
@@
 $EndComp
 $Comp
-L antmicroMicrocontrollers:XC7A100T-FGG484 U14
+L artix-dc-scm:XC7A100T-FGG484 U14
 U 6 1 605660E8
 P 7950 9150
 F 0 "U14" H 7921 9203 50  0000 R CNN
 F 1 "XC7A100T-FGG484" H 7921 9112 50  0000 R CNN
-F 2 "antmicro-footprints:Xilinx_FGG484" H 7650 9150 50  0001 C CNN
+F 2 "artix-dc-scm-footprints:Xilinx_FGG484" H 7650 9150 50  0001 C CNN
 F 3 "" H 7650 9150 50  0000 C CNN
 	6    7950 9150
@@
 	11100 9350 10650 9350
 $Comp
-L antmicroResistors0402:R_100R_0402 R86
+L artix-dc-scm:R_100R_0402 R86
 U 1 1 60A2E489
 P 10000 8550
 F 0 "R86" V 9955 8620 60  0000 L CNN
 F 1 "R_100R_0402" H 10000 8400 60  0001 C CNN
-F 2 "antmicro-footprints:0402-res" H 10200 8750 60  0001 L CNN
+F 2 "artix-dc-scm-footprints:0402-res" H 10200 8750 60  0001 L CNN
 F 3 "" H 10000 8550 50  0001 C CNN
 F 4 "BOURNS" H 10200 8950 60  0001 L CNN "Manufacturer"
@@
 	10000 8400 10000 8150
 $Comp
-L antmicroResistors0402:R_200R_0402 R88
+L artix-dc-scm:R_200R_0402 R88
 U 1 1 60B66864
 P 10650 8550
 F 0 "R88" V 10605 8620 60  0000 L CNN
 F 1 "R_200R_0402" H 10650 8400 60  0001 C CNN
-F 2 "antmicro-footprints:0402-res" H 10850 8750 60  0001 L CNN
+F 2 "artix-dc-scm-footprints:0402-res" H 10850 8750 60  0001 L CNN
 F 3 "" H 10650 8550 50  0001 C CNN
 F 4 "YAGEO" H 10850 8950 60  0001 L CNN "Manufacturer"
@@
 $EndComp
 $Comp
-L antmicroResistors0402:R_4k7_0402 R89
+L artix-dc-scm:R_4k7_0402 R89
 U 1 1 60B67874
 P 10800 8850
 F 0 "R89" V 10755 8920 60  0000 L CNN
 F 1 "R_4k7_0402" H 10800 8700 60  0001 C CNN
-F 2 "antmicro-footprints:0402-res" H 11000 9050 60  0001 L CNN
+F 2 "artix-dc-scm-footprints:0402-res" H 11000 9050 60  0001 L CNN
 F 3 "" H 10800 8850 50  0001 C CNN
 F 4 "PANASONIC_ELECTRONIC_COMPONENTS" H 11000 9250 60  0001 L CNN "Manufacturer"
@@
 Connection ~ 10800 9550
 $Comp
-L antmicroResistors0402:R_4k7_0402 R90
+L artix-dc-scm:R_4k7_0402 R90
 U 1 1 60BCAC0A
 P 10950 8550
 F 0 "R90" V 10905 8620 60  0000 L CNN
 F 1 "R_4k7_0402" H 10950 8400 60  0001 C CNN
-F 2 "antmicro-footprints:0402-res" H 11150 8750 60  0001 L CNN
+F 2 "artix-dc-scm-footprints:0402-res" H 11150 8750 60  0001 L CNN
 F 3 "" H 10950 8550 50  0001 C CNN
 F 4 "PANASONIC_ELECTRONIC_COMPONENTS" H 11150 8950 60  0001 L CNN "Manufacturer"
@@
 	10800 8150 10800 8300
 $Comp
-L antmicroResistors0402:R_4k7_0402 R85
+L artix-dc-scm:R_4k7_0402 R85
 U 1 1 60C6C820
 P 9750 9750
 F 0 "R85" H 9750 9537 60  0000 C CNN
 F 1 "R_4k7_0402" H 9750 9600 60  0001 C CNN
-F 2 "antmicro-footprints:0402-res" H 9950 9950 60  0001 L CNN
+F 2 "artix-dc-scm-footprints:0402-res" H 9950 9950 60  0001 L CNN
 F 3 "" H 9750 9750 50  0001 C CNN
 F 4 "PANASONIC_ELECTRONIC_COMPONENTS" H 9950 10150 60  0001 L CNN "Manufacturer"
@@
 	9900 9750 10050 9750
 $Comp
-L antmicroResistors0402:R_100R_0402 R87
+L artix-dc-scm:R_100R_0402 R87
 U 1 1 60D065C0
 P 10000 9000
 F 0 "R87" V 9955 9070 60  0000 L CNN
 F 1 "R_100R_0402" H 10000 8850 60  0001 C CNN
-F 2 "antmicro-footprints:0402-res" H 10200 9200 60  0001 L CNN
+F 2 "artix-dc-scm-footprints:0402-res" H 10200 9200 60  0001 L CNN
 F 3 "" H 10000 9000 50  0001 C CNN
 F 4 "BOURNS" H 10200 9400 60  0001 L CNN "Manufacturer"
@@
 $EndComp
 $Comp
-L power:GND #PWR085
+L artix-dc-scm:GND #PWR085
 U 1 1 60D0D551
 P 10000 9150
@@
 $EndComp
 $Comp
-L antmicroPushbuttonSwitches:KMR2 S1
+L artix-dc-scm:KMR2 S1
 U 1 1 60DA2AC9
 P 10900 10100
 F 0 "S1" V 10854 10238 50  0000 L CNN
 F 1 "KMR2" V 10945 10238 50  0000 L CNN
-F 2 "antmicro-footprints:SW_SPST_4.2x2.8" H 11100 10300 50  0001 L CNN
+F 2 "artix-dc-scm-footprints:SW_SPST_4.2x2.8" H 11100 10300 50  0001 L CNN
 F 3 "http://www.farnell.com/datasheets/2631211.pdf" H 11100 10400 60  0001 L CNN
 F 4 "KMR211NGLFS" H 11096 10493 60  0001 L CNN "MPN"
@@
 Connection ~ 10800 10250
 $Comp
-L power:GND #PWR086
+L artix-dc-scm:GND #PWR086
 U 1 1 60E5F880
 P 10800 10450
@@
 	9450 10650 9450 10850
 $Comp
-L power:GND #PWR084
+L artix-dc-scm:GND #PWR084
 U 1 1 60E9E149
 P 9450 10850
@@
 VCC3V3
 $Comp
-L power:GND #PWR081
+L artix-dc-scm:GND #PWR081
 U 1 1 612D9DD9
 P 6250 10200
@@
 $EndComp
 $Comp
-L power:GND #PWR080
+L artix-dc-scm:GND #PWR080
 U 1 1 612DAB50
 P 6250 9900
@@
 $EndComp
 $Comp
-L antmicroCapacitorsmisc:C_47u_1210 C178
+L artix-dc-scm:C_47u_1210 C178
 U 1 1 6143B808
 P 9450 7800
 F 0 "C178" H 9565 7845 60  0000 L CNN
 F 1 "C_47u_1210" H 9450 7650 60  0001 C CNN
-F 2 "antmicro-footprints:1210-cap" H 9650 8000 60  0001 L CNN
+F 2 "artix-dc-scm-footprints:1210-cap" H 9650 8000 60  0001 L CNN
 F 3 "" H 9450 7800 50  0001 C CNN
 F 4 "KEMET" H 9650 8200 60  0001 L CNN "Manufacturer"
@@
 	9450 7550 9050 7550
 $Comp
-L power:GND #PWR083
+L artix-dc-scm:GND #PWR083
 U 1 1 6148AC43
 P 9450 7950
@@
 	9450 10350 9450 10550
 $Comp
-L antmicroResistors0402:R_0R_0402 R81
+L artix-dc-scm:R_0R_0402 R81
 U 1 1 648CDBE7
 P 6575 9775
 F 0 "R81" H 6575 9988 60  0000 C CNN
 F 1 "R_0R_0402" H 6575 9625 60  0001 C CNN
-F 2 "antmicro-footprints:0402-res" H 6775 9975 60  0001 L CNN
+F 2 "artix-dc-scm-footprints:0402-res" H 6775 9975 60  0001 L CNN
 F 3 "" H 6575 9775 50  0001 C CNN
 F 4 "PANASONIC" H 6775 10175 60  0001 L CNN "Manufacturer"
@@
 $EndComp
 $Comp
-L antmicroResistors0402:R_0R_0402 R82
+L artix-dc-scm:R_0R_0402 R82
 U 1 1 648CE50A
 P 6575 9900
 F 0 "R82" H 6575 10113 60  0000 C CNN
 F 1 "R_0R_0402" H 6575 9750 60  0001 C CNN
-F 2 "antmicro-footprints:0402-res" H 6775 10100 60  0001 L CNN
+F 2 "artix-dc-scm-footprints:0402-res" H 6775 10100 60  0001 L CNN
 F 3 "" H 6575 9900 50  0001 C CNN
 F 4 "PANASONIC" H 6775 10300 60  0001 L CNN "Manufacturer"
@@
 $EndComp
 $Comp
-L antmicroResistors0402:R_0R_0402 R83
+L artix-dc-scm:R_0R_0402 R83
 U 1 1 648D070F
 P 6575 10075
 F 0 "R83" H 6575 10288 60  0000 C CNN
 F 1 "R_0R_0402" H 6575 9925 60  0001 C CNN
-F 2 "antmicro-footprints:0402-res" H 6775 10275 60  0001 L CNN
+F 2 "artix-dc-scm-footprints:0402-res" H 6775 10275 60  0001 L CNN
 F 3 "" H 6575 10075 50  0001 C CNN
 F 4 "PANASONIC" H 6775 10475 60  0001 L CNN "Manufacturer"
@@
 $EndComp
 $Comp
-L antmicroResistors0402:R_0R_0402 R84
+L artix-dc-scm:R_0R_0402 R84
 U 1 1 648D0718
 P 6575 10200
 F 0 "R84" H 6575 10413 60  0000 C CNN
 F 1 "R_0R_0402" H 6575 10050 60  0001 C CNN
-F 2 "antmicro-footprints:0402-res" H 6775 10400 60  0001 L CNN
+F 2 "artix-dc-scm-footprints:0402-res" H 6775 10400 60  0001 L CNN
 F 3 "" H 6575 10200 50  0001 C CNN
 F 4 "PANASONIC" H 6775 10600 60  0001 L CNN "Manufacturer"
@@
 	6775 10075 6725 10075
 $Comp
-L antmicroRectangularConnectorsHeadersMalePins:62000311121 J13
+L artix-dc-scm:62000311121 J13
 U 1 1 649873F1
 P 6525 10500
 F 0 "J13" H 6583 10733 50  0000 C CNN
 F 1 "62000311121" H 6575 10300 50  0001 C CNN
-F 2 "antmicro-footprints:62000311121" H 6625 10750 60  0001 L CNN
+F 2 "artix-dc-scm-footprints:62000311121" H 6625 10750 60  0001 L CNN
 F 3 "https://www.we-online.com/catalog/datasheet/62000311121.pdf" H 6725 10800 60  0001 L CNN
 F 4 "62000421121" H 6725 11000 60  0001 L CNN "MPN"
@@
 	6800 10400 6675 10400
 $Comp
-L power:GND #PWR082
+L artix-dc-scm:GND #PWR082
 U 1 1 649B5B60
 P 6825 10600
