File: ddr3.sch (KiCad schematic (older format))
At the start: 35 parts, among them U7 AS4C256M16D3, U8 TPS51200DRC

Commit message: Swapped RAS and CAS connection
Parts:
- added C?: C_1n_0402, antmicro-footprints:0402-res, symbol antmicroCapacitors0402:C_1n_0402
Connections:
- wire segments 329 -> 333
Other:
- moved on the sheet: C42, C44, R57, R58
Changed lines of the file:
@@
 Text GLabel 3650 5125 0    50   Input ~ 0
 DDR3_CS
+Text GLabel 3650 5325 0    50   Input ~ 0
+DDR3_CAS
 Text GLabel 3650 5225 0    50   Input ~ 0
-DDR3_CAS
-Text GLabel 3650 5325 0    50   Input ~ 0
 DDR3_RAS
 Text GLabel 3650 5425 0    50   Input ~ 0
@@
 Wire Wire Line
 	6925 8650 7350 8650
-$Comp
-L artix-dc-scm:GND #PWR037
-U 1 1 618D515B
-P 5825 9075
-F 0 "#PWR037" H 5825 8825 50  0001 C CNN
-F 1 "GND" H 5830 8902 50  0000 C CNN
-F 2 "" H 5825 9075 50  0001 C CNN
-F 3 "" H 5825 9075 50  0001 C CNN
-	1    5825 9075
-	1    0    0    -1
-$EndComp
-Text GLabel 6900 8950 0    50   Output ~ 0
+Text GLabel 7000 8950 0    50   Output ~ 0
 DDR3_VREF
 Wire Wire Line
-	6900 8950 6950 8950
+	7000 8950 7050 8950
 $Comp
 L artix-dc-scm:GND #PWR039
@@
 Wire Wire Line
 	8500 8950 8350 8950
-Connection ~ 7250 8950
-Wire Wire Line
-	7250 8950 7350 8950
+Connection ~ 7300 8950
+Wire Wire Line
+	7300 8950 7350 8950
 Text Label 8850 8750 2    50   ~ 0
 DDR3_VTT
@@
 L artix-dc-scm:R_10k_0402 R57
 U 1 1 609FEB6C
-P 6125 8850
-F 0 "R57" H 6175 8775 60  0000 L CNN
-F 1 "R_10k_0402" H 6125 8700 60  0001 C CNN
-F 2 "artix-dc-scm-footprints:0402-res" H 6325 9050 60  0001 L CNN
-F 3 "" H 6125 8850 50  0001 C CNN
-F 4 "VISHAY" H 6325 9250 60  0001 L CNN "Manufacturer"
-F 5 "CRCW040210K0FKEDHP" H 6325 9150 60  0001 L CNN "MPN"
-F 6 "10k" H 5875 8900 50  0000 L CNN "Val"
-	1    6125 8850
-	-1   0    0    1
+P 6175 9175
+F 0 "R57" H 6225 9100 60  0000 L CNN
+F 1 "R_10k_0402" H 6175 9025 60  0001 C CNN
+F 2 "artix-dc-scm-footprints:0402-res" H 6375 9375 60  0001 L CNN
+F 3 "" H 6175 9175 50  0001 C CNN
+F 4 "VISHAY" H 6375 9575 60  0001 L CNN "Manufacturer"
+F 5 "CRCW040210K0FKEDHP" H 6375 9475 60  0001 L CNN "MPN"
+F 6 "10k" H 5925 9225 50  0000 L CNN "Val"
+	1    6175 9175
+	0    -1   -1   0
 $EndComp
 Wire Wire Line
@@
 Wire Wire Line
 	8400 7025 8875 7025
-Text GLabel 6325 8000 0    50   Input ~ 0
+Text GLabel 6100 8000 0    50   Input ~ 0
 VCC1V35
 Wire Wire Line
-	6400 8000 6325 8000
+	6175 8000 6100 8000
 Text GLabel 9325 8200 2    50   Input ~ 0
 VCC3V3
@@
 VLDOIN
 Wire Wire Line
-	6400 8850 7350 8850
-Connection ~ 6400 8850
-Wire Wire Line
-	6950 9400 7100 9400
-Connection ~ 6950 8950
-Wire Wire Line
-	6950 8950 7250 8950
+	7050 9450 7200 9450
+Connection ~ 7050 8950
+Wire Wire Line
+	7050 8950 7300 8950
 $Comp
 L artix-dc-scm:GND #PWR038
 U 1 1 6132157D
-P 7100 9550
-F 0 "#PWR038" H 7100 9300 50  0001 C CNN
-F 1 "GND" H 7105 9377 50  0000 C CNN
-F 2 "" H 7100 9550 50  0001 C CNN
-F 3 "" H 7100 9550 50  0001 C CNN
-	1    7100 9550
-	1    0    0    -1
-$EndComp
-Wire Wire Line
-	7100 9550 7100 9400
-Connection ~ 7100 9400
-Wire Wire Line
-	7100 9400 7250 9400
-Wire Wire Line
-	6950 8950 6950 9025
-Wire Wire Line
-	7250 8950 7250 9025
-Wire Wire Line
-	7250 9325 7250 9400
-Wire Wire Line
-	6950 9325 6950 9400
-Wire Wire Line
-	6400 8850 6275 8850
-Wire Wire Line
-	6400 8000 6400 8250
+P 7200 9550
+F 0 "#PWR038" H 7200 9300 50  0001 C CNN
+F 1 "GND" H 7205 9377 50  0000 C CNN
+F 2 "" H 7200 9550 50  0001 C CNN
+F 3 "" H 7200 9550 50  0001 C CNN
+	1    7200 9550
+	1    0    0    -1
+$EndComp
+Wire Wire Line
+	7200 9550 7200 9450
+Connection ~ 7200 9450
+Wire Wire Line
+	7200 9450 7300 9450
+Wire Wire Line
+	7050 8950 7050 9025
+Wire Wire Line
+	7300 8950 7300 9025
+Wire Wire Line
+	7300 9325 7300 9450
+Wire Wire Line
+	7050 9325 7050 9450
+Wire Wire Line
+	6175 8000 6175 8250
 $Comp
 L artix-dc-scm:R_10k_0402 R58
 U 1 1 614307C1
-P 6400 8400
-F 0 "R58" V 6355 8470 60  0000 L CNN
-F 1 "R_10k_0402" H 6400 8250 60  0001 C CNN
-F 2 "artix-dc-scm-footprints:0402-res" H 6600 8600 60  0001 L CNN
-F 3 "" H 6400 8400 50  0001 C CNN
-F 4 "VISHAY" H 6600 8800 60  0001 L CNN "Manufacturer"
-F 5 "CRCW040210K0FKEDHP" H 6600 8700 60  0001 L CNN "MPN"
-F 6 "10k" V 6453 8470 50  0000 L CNN "Val"
-	1    6400 8400
+P 6175 8400
+F 0 "R58" V 6130 8470 60  0000 L CNN
+F 1 "R_10k_0402" H 6175 8250 60  0001 C CNN
+F 2 "artix-dc-scm-footprints:0402-res" H 6375 8600 60  0001 L CNN
+F 3 "" H 6175 8400 50  0001 C CNN
+F 4 "VISHAY" H 6375 8800 60  0001 L CNN "Manufacturer"
+F 5 "CRCW040210K0FKEDHP" H 6375 8700 60  0001 L CNN "MPN"
+F 6 "10k" V 6228 8470 50  0000 L CNN "Val"
+	1    6175 8400
 	0    1    1    0
 $EndComp
-Wire Wire Line
-	6400 8550 6400 8850
 Wire Wire Line
 	7850 7025 8100 7025
@@
 Wire Wire Line
 	7000 7025 7350 7025
-Wire Wire Line
-	5975 8850 5825 8850
-Wire Wire Line
-	5825 8850 5825 9075
 Wire Wire Line
 	6925 8000 6925 8225
@@
 L artix-dc-scm:C_100n_0402 C?
 U 1 1 62867A2A
-P 6950 9175
+P 7050 9175
 AR Path="/62867A2A" Ref="C?"  Part="1"
 AR Path="/5FD8EBC2/62867A2A" Ref="C42"  Part="1"
-F 0 "C42" H 6975 9275 60  0000 L CNN
-F 1 "C_100n_0402" H 6950 9025 60  0001 C CNN
-F 2 "artix-dc-scm-footprints:0402-cap" H 7150 9375 60  0001 L CNN
-F 3 "" H 6950 9175 50  0001 C CNN
-F 4 "Walsin" H 7150 9575 60  0001 L CNN "Manufacturer"
-F 5 "0402X104K6R3CT" H 7150 9475 60  0001 L CNN "MPN"
-F 6 "100n" H 6975 9075 50  0000 L CNN "Val"
-	1    6950 9175
+F 0 "C42" H 7075 9275 60  0000 L CNN
+F 1 "C_100n_0402" H 7050 9025 60  0001 C CNN
+F 2 "artix-dc-scm-footprints:0402-cap" H 7250 9375 60  0001 L CNN
+F 3 "" H 7050 9175 50  0001 C CNN
+F 4 "Walsin" H 7250 9575 60  0001 L CNN "Manufacturer"
+F 5 "0402X104K6R3CT" H 7250 9475 60  0001 L CNN "MPN"
+F 6 "100n" H 7075 9075 50  0000 L CNN "Val"
+	1    7050 9175
 	1    0    0    -1
 $EndComp
@@
 L artix-dc-scm:C_100n_0402 C?
 U 1 1 62867ED9
-P 7250 9175
+P 7300 9175
 AR Path="/62867ED9" Ref="C?"  Part="1"
 AR Path="/5FD8EBC2/62867ED9" Ref="C44"  Part="1"
-F 0 "C44" H 7275 9275 60  0000 L CNN
-F 1 "C_100n_0402" H 7250 9025 60  0001 C CNN
-F 2 "artix-dc-scm-footprints:0402-cap" H 7450 9375 60  0001 L CNN
-F 3 "" H 7250 9175 50  0001 C CNN
-F 4 "Walsin" H 7450 9575 60  0001 L CNN "Manufacturer"
-F 5 "0402X104K6R3CT" H 7450 9475 60  0001 L CNN "MPN"
-F 6 "100n" H 7275 9075 50  0000 L CNN "Val"
-	1    7250 9175
+F 0 "C44" H 7325 9275 60  0000 L CNN
+F 1 "C_100n_0402" H 7300 9025 60  0001 C CNN
+F 2 "artix-dc-scm-footprints:0402-cap" H 7500 9375 60  0001 L CNN
+F 3 "" H 7300 9175 50  0001 C CNN
+F 4 "Walsin" H 7500 9575 60  0001 L CNN "Manufacturer"
+F 5 "0402X104K6R3CT" H 7500 9475 60  0001 L CNN "MPN"
+F 6 "100n" H 7325 9075 50  0000 L CNN "Val"
+	1    7300 9175
 	1    0    0    -1
 $EndComp
@@
 Text GLabel 4425 7675 0    50   UnSpc ~ 0
 DDR3_A9
+$Comp
+L antmicroCapacitors0402:C_1n_0402 C?
+U 1 1 6033B485
+P 6400 9175
+F 0 "C?" H 6515 9220 60  0000 L CNN
+F 1 "C_1n_0402" H 6400 9025 60  0001 C CNN
+F 2 "antmicro-footprints:0402-res" H 6600 9375 60  0001 L CNN
+F 3 "" H 6400 9175 50  0001 C CNN
+F 4 "YAGEO" H 6600 9575 60  0001 L CNN "Manufacturer"
+F 5 "CC0402KRX7R9BB102" H 6600 9475 60  0001 L CNN "MPN"
+F 6 "1n" H 6515 9122 50  0000 L CNN "Val"
+	1    6400 9175
+	1    0    0    -1
+$EndComp
+Wire Wire Line
+	6400 9325 6400 9450
+$Comp
+L artix-dc-scm:GND #PWR?
+U 1 1 603993AB
+P 6400 9550
+F 0 "#PWR?" H 6400 9300 50  0001 C CNN
+F 1 "GND" H 6405 9377 50  0000 C CNN
+F 2 "" H 6400 9550 50  0001 C CNN
+F 3 "" H 6400 9550 50  0001 C CNN
+	1    6400 9550
+	1    0    0    -1
+$EndComp
+Wire Wire Line
+	6175 8850 6175 9025
+Wire Wire Line
+	6175 9325 6175 9450
+Wire Wire Line
+	6175 9450 6400 9450
+Connection ~ 6400 9450
+Wire Wire Line
+	6400 9450 6400 9550
+Wire Wire Line
+	6175 8850 6400 8850
+Wire Wire Line
+	6400 9025 6400 8850
+Connection ~ 6400 8850
+Wire Wire Line
+	6400 8850 7350 8850
+Wire Wire Line
+	6175 8850 6175 8550
+Connection ~ 6175 8850
 $EndSCHEMATC
