File: fpga-power-supply.sch (KiCad schematic (older format))
At the start: 88 parts

Commit message: Minor changes to FPGA
Parts:
- added C? (x3): C_10u_0402, antmicro-footprints:0402-cap, symbol antmicroCapacitors0402:C_10u_0402
- added C?: C_1u_0402, antmicro-footprints:0402-cap, symbol antmicroCapacitors0402:C_1u_0402
- added C?: C_470n_0402, antmicro-footprints:0402-cap, symbol antmicroCapacitors0402:C_470n_0402
- added C?: C_100n_0402, antmicro-footprints:0402-cap, symbol antmicroCapacitors0402:C_100n_0402
- added FB?: BLM18PG121SN1D, antmicro-footprints:0603-res, symbol antmicroFerriteBeadsandChips:BLM18PG121SN1D
- added L?: 10uH, antmicro-footprints:0805-res, symbol antmicroFixedInductors:10uH
- added U?: REF3012AIDBZT, antmicro-footprints:SOT-23-3, symbol antmicroPMICPowerDistributionSwitchesLoadDrivers:REF3012AIDBZT
Connections:
- net labels added: AVCC3V3, VCC3V3, XADCVREF
- wire segments 476 -> 493
Changed lines of the file:
@@
 Text Notes 11700 2150 0    118  ~ 0
 VCCINT decoupling
+Text GLabel 15350 9100 3    50   Input ~ 0
+XADCGND
+Text GLabel 15350 8800 1    50   Input ~ 0
+XADCVREF
+Text GLabel 12300 9150 3    50   Input ~ 0
+XADCGND
+Text GLabel 12300 8850 1    50   Input ~ 0
+AVCC3V3
+$Comp
+L antmicroCapacitors0402:C_100n_0402 C?
+U 1 1 645D96CD
+P 12300 9000
+F 0 "C?" H 12415 9045 60  0000 L CNN
+F 1 "C_100n_0402" H 12300 8850 60  0001 C CNN
+F 2 "antmicro-footprints:0402-cap" H 12500 9200 60  0001 L CNN
+F 3 "" H 12300 9000 50  0001 C CNN
+F 4 "Walsin" H 12500 9400 60  0001 L CNN "Manufacturer"
+F 5 "0402X104K6R3CT" H 12500 9300 60  0001 L CNN "MPN"
+F 6 "100n" H 12415 8947 50  0000 L CNN "Val"
+	1    12300 9000
+	1    0    0    -1
+$EndComp
+$Comp
+L antmicroCapacitors0402:C_10u_0402 C?
+U 1 1 645D82F3
+P 15350 8950
+F 0 "C?" H 15465 8995 60  0000 L CNN
+F 1 "C_10u_0402" H 15350 8800 60  0001 C CNN
+F 2 "antmicro-footprints:0402-cap" H 15550 9150 60  0001 L CNN
+F 3 "" H 15350 8950 50  0001 C CNN
+F 4 "MURATA" H 15550 9350 60  0001 L CNN "Manufacturer"
+F 5 "GRM155R60J106ME44D" H 15550 9250 60  0001 L CNN "MPN"
+F 6 "10u" H 15465 8897 50  0000 L CNN "Val"
+	1    15350 8950
+	1    0    0    -1
+$EndComp
+Text GLabel 14450 8975 2    50   Input ~ 0
+XADCVREF
+Wire Wire Line
+	14175 8975 14450 8975
+Wire Wire Line
+	13275 9125 13200 9125
+Text GLabel 13200 9125 0    50   Input ~ 0
+XADCGND
+Wire Wire Line
+	12825 8900 12825 8975
+Text GLabel 12825 8900 1    50   Input ~ 0
+AVCC3V3
+Wire Wire Line
+	13275 8975 12825 8975
+$Comp
+L antmicroPMICPowerDistributionSwitchesLoadDrivers:REF3012AIDBZT U?
+U 1 1 643B2A61
+P 13975 8975
+F 0 "U?" H 13725 9190 50  0000 C CNN
+F 1 "REF3012AIDBZT" H 13725 9099 50  0000 C CNN
+F 2 "antmicro-footprints:SOT-23-3" H 14125 9275 50  0001 L BNN
+F 3 "" H 14125 9375 50  0001 L BNN
+	1    13975 8975
+	1    0    0    -1
+$EndComp
+Text GLabel 14425 7650 2    50   Input ~ 0
+AVCC3V3
+Text GLabel 12800 7550 1    50   Input ~ 0
+VCC3V3
+$Comp
+L power:GND #PWR?
+U 1 1 642F2B49
+P 13025 8150
+F 0 "#PWR?" H 13025 7900 50  0001 C CNN
+F 1 "GND" H 13030 7977 50  0000 C CNN
+F 2 "" H 13025 8150 50  0001 C CNN
+F 3 "" H 13025 8150 50  0001 C CNN
+	1    13025 8150
+	1    0    0    -1
+$EndComp
+Wire Wire Line
+	13025 7950 13025 8150
+Wire Wire Line
+	12800 7650 12800 7550
+Wire Wire Line
+	14100 7650 14425 7650
+Connection ~ 14100 7650
+$Comp
+L antmicroCapacitors0402:C_470n_0402 C?
+U 1 1 64284146
+P 14100 7800
+F 0 "C?" H 14215 7845 60  0000 L CNN
+F 1 "C_470n_0402" H 14100 7650 60  0001 C CNN
+F 2 "antmicro-footprints:0402-cap" H 14300 8000 60  0001 L CNN
+F 3 "" H 14100 7800 50  0001 C CNN
+F 4 "TDK" H 14300 8200 60  0001 L CNN "Manufacturer"
+F 5 "C1005X5R1E474M050BB" H 14300 8100 60  0001 L CNN "MPN"
+F 6 "470n" H 14215 7747 50  0000 L CNN "Val"
+	1    14100 7800
+	1    0    0    -1
+$EndComp
+Wire Wire Line
+	13775 7650 14100 7650
+Connection ~ 13775 7650
+Wire Wire Line
+	14100 7950 13775 7950
+Connection ~ 13775 7950
+$Comp
+L antmicroCapacitors0402:C_1u_0402 C?
+U 1 1 64282C33
+P 13775 7800
+F 0 "C?" H 13660 7755 60  0000 R CNN
+F 1 "C_1u_0402" H 13775 7650 60  0001 C CNN
+F 2 "antmicro-footprints:0402-cap" H 13975 8000 60  0001 L CNN
+F 3 "" H 13775 7800 50  0001 C CNN
+F 4 "TDK" H 13975 8200 60  0001 L CNN "Manufacturer"
+F 5 "C1005X6S1A105K050BC" H 13975 8100 60  0001 L CNN "MPN"
+F 6 "1u" H 13660 7853 50  0000 R CNN "Val"
+	1    13775 7800
+	-1   0    0    1
+$EndComp
+Wire Wire Line
+	13500 7650 13775 7650
+Wire Wire Line
+	13400 7650 13500 7650
+Connection ~ 13500 7650
+Wire Wire Line
+	13775 7950 13500 7950
+Wire Wire Line
+	13500 7950 13025 7950
+Connection ~ 13500 7950
+$Comp
+L antmicroCapacitors0402:C_10u_0402 C?
+U 1 1 6427ABFA
+P 13500 7800
+F 0 "C?" H 13385 7755 60  0000 R CNN
+F 1 "C_10u_0402" H 13500 7650 60  0001 C CNN
+F 2 "antmicro-footprints:0402-cap" H 13700 8000 60  0001 L CNN
+F 3 "" H 13500 7800 50  0001 C CNN
+F 4 "MURATA" H 13700 8200 60  0001 L CNN "Manufacturer"
+F 5 "GRM155R60J106ME44D" H 13700 8100 60  0001 L CNN "MPN"
+F 6 "10u" H 13385 7853 50  0000 R CNN "Val"
+	1    13500 7800
+	-1   0    0    1
+$EndComp
+Wire Wire Line
+	13025 7650 12800 7650
+Wire Wire Line
+	13100 7650 13025 7650
+Connection ~ 13025 7650
+Connection ~ 13025 7950
+$Comp
+L antmicroCapacitors0402:C_10u_0402 C?
+U 1 1 642799BF
+P 13025 7800
+F 0 "C?" H 12910 7755 60  0000 R CNN
+F 1 "C_10u_0402" H 13025 7650 60  0001 C CNN
+F 2 "antmicro-footprints:0402-cap" H 13225 8000 60  0001 L CNN
+F 3 "" H 13025 7800 50  0001 C CNN
+F 4 "MURATA" H 13225 8200 60  0001 L CNN "Manufacturer"
+F 5 "GRM155R60J106ME44D" H 13225 8100 60  0001 L CNN "MPN"
+F 6 "10u" H 12910 7853 50  0000 R CNN "Val"
+	1    13025 7800
+	-1   0    0    1
+$EndComp
+$Comp
+L antmicroFixedInductors:10uH L?
+U 1 1 64278577
+P 13250 7650
+F 0 "L?" H 13250 7864 60  0000 C CNN
+F 1 "10uH" H 13250 7758 60  0000 C CNN
+F 2 "antmicro-footprints:0805-res" H 13300 7500 60  0001 C CNN
+F 3 "" H 13305 7680 60  0001 C CNN
+F 4 "TDK" H 13250 7550 50  0001 C CNN "Manufacturer"
+F 5 "MLZ2012N100LT000" H 13200 7600 50  0001 C CNN "MPN"
+	1    13250 7650
+	1    0    0    -1
+$EndComp
+Text GLabel 13200 9500 0    50   Input ~ 0
+XADCGND
+$Comp
+L power:GND #PWR?
+U 1 1 64669A59
+P 13875 9500
+F 0 "#PWR?" H 13875 9250 50  0001 C CNN
+F 1 "GND" V 13880 9372 50  0000 R CNN
+F 2 "" H 13875 9500 50  0001 C CNN
+F 3 "" H 13875 9500 50  0001 C CNN
+	1    13875 9500
+	0    -1   -1   0
+$EndComp
+$Comp
+L antmicroFerriteBeadsandChips:BLM18PG121SN1D FB?
+U 1 1 6466A4B3
+P 13500 9500
+F 0 "FB?" H 13500 9787 60  0000 C CNN
+F 1 "BLM18PG121SN1D" H 13500 9681 60  0000 C CNN
+F 2 "antmicro-footprints:0603-res" H 13700 9700 60  0001 L CNN
+F 3 "https://www.murata.com/en-us/products/productdata/8796738650142/ENFA0003.pdf" H 13700 9800 60  0001 L CNN
+F 4 "BLM18PG121SN1D" H 13700 10000 60  0001 L CNN "MPN"
+F 5 "Murata Electronics North America" H 13700 10600 60  0001 L CNN "Manufacturer"
+	1    13500 9500
+	1    0    0    -1
+$EndComp
+Wire Wire Line
+	13200 9500 13300 9500
+Wire Wire Line
+	13700 9500 13875 9500
 $EndSCHEMATC

Commit message: FPGA supplies update
Parts:
- removed C? (x3): C_10u_0402, antmicro-footprints:0402-cap, symbol antmicroCapacitors0402:C_10u_0402
- removed C?: C_1u_0402, antmicro-footprints:0402-cap, symbol antmicroCapacitors0402:C_1u_0402
- removed C?: C_470n_0402, antmicro-footprints:0402-cap, symbol antmicroCapacitors0402:C_470n_0402
- removed C?: C_100n_0402, antmicro-footprints:0402-cap, symbol antmicroCapacitors0402:C_100n_0402
- removed FB?: BLM18PG121SN1D, antmicro-footprints:0603-res, symbol antmicroFerriteBeadsandChips:BLM18PG121SN1D
- removed L?: 10uH, antmicro-footprints:0805-res, symbol antmicroFixedInductors:10uH
- removed U?: REF3012AIDBZT, antmicro-footprints:SOT-23-3, symbol antmicroPMICPowerDistributionSwitchesLoadDrivers:REF3012AIDBZT
Connections:
- net labels added: VCC1V0
- net labels removed: AVCC3V3, VCC3V3, VCCBRAM, VCCINT, XADCVREF
- wire segments 493 -> 476
Other:
- note added: "VCCAUX decoupling"
Changed lines of the file:
@@
 	7750 3600 7600 3600
 Text GLabel 7600 3600 0    50   Input ~ 0
-XADC1V8
+VCC1V8
 Text GLabel 4650 3800 1    50   Input ~ 0
 XADC1V8
@@
 	4650 4400 4650 4500
 Connection ~ 4650 4400
-Text GLabel 7600 3500 0    50   Input ~ 0
-XADCGND
 Wire Wire Line
 	7750 3500 7600 3500
@@
 	7600 3900 7600 3800
 Text GLabel 7400 3800 0    50   Input ~ 0
-VCCBRAM
+VCC1V0
 Wire Wire Line
 	7600 3800 7400 3800
 Connection ~ 7600 3800
 Text GLabel 9900 2600 1    50   Input ~ 0
-VCCINT
+VCC1V0
 $Comp
 L antmicroCapacitorsmisc:C_100u_1210 C?
@@
 BRAM decoupling
 Text GLabel 5500 4300 1    50   Input ~ 0
-VCCINT
+VCC1V0
 $Comp
 L antmicroCapacitorspol:C_330u_KEMET_D C?
@@
 Connection ~ 11500 4100
 Text GLabel 12050 2600 1    50   Input ~ 0
-VCCINT
+VCC1V0
 Text GLabel 11500 3900 1    50   Input ~ 0
-VCCINT
+VCC1V0
 $Comp
 L antmicroCapacitorspol:C_680u_KEMET_D C?
@@
 	11000 2800 11000 2600
 Text GLabel 11000 2600 1    50   Input ~ 0
-VCCINT
+VCC1V0
 Text Notes 10550 2800 3    50   ~ 0
 populate on \n
 Text Notes 11700 2150 0    118  ~ 0
 VCCINT decoupling
-Text GLabel 15350 9100 3    50   Input ~ 0
-XADCGND
-Text GLabel 15350 8800 1    50   Input ~ 0
-XADCVREF
-Text GLabel 12300 9150 3    50   Input ~ 0
-XADCGND
-Text GLabel 12300 8850 1    50   Input ~ 0
-AVCC3V3
-$Comp
-L antmicroCapacitors0402:C_100n_0402 C?
-U 1 1 645D96CD
-P 12300 9000
-F 0 "C?" H 12415 9045 60  0000 L CNN
-F 1 "C_100n_0402" H 12300 8850 60  0001 C CNN
-F 2 "antmicro-footprints:0402-cap" H 12500 9200 60  0001 L CNN
-F 3 "" H 12300 9000 50  0001 C CNN
-F 4 "Walsin" H 12500 9400 60  0001 L CNN "Manufacturer"
-F 5 "0402X104K6R3CT" H 12500 9300 60  0001 L CNN "MPN"
-F 6 "100n" H 12415 8947 50  0000 L CNN "Val"
-	1    12300 9000
-	1    0    0    -1
-$EndComp
-$Comp
-L antmicroCapacitors0402:C_10u_0402 C?
-U 1 1 645D82F3
-P 15350 8950
-F 0 "C?" H 15465 8995 60  0000 L CNN
-F 1 "C_10u_0402" H 15350 8800 60  0001 C CNN
-F 2 "antmicro-footprints:0402-cap" H 15550 9150 60  0001 L CNN
-F 3 "" H 15350 8950 50  0001 C CNN
-F 4 "MURATA" H 15550 9350 60  0001 L CNN "Manufacturer"
-F 5 "GRM155R60J106ME44D" H 15550 9250 60  0001 L CNN "MPN"
-F 6 "10u" H 15465 8897 50  0000 L CNN "Val"
-	1    15350 8950
-	1    0    0    -1
-$EndComp
-Text GLabel 14450 8975 2    50   Input ~ 0
-XADCVREF
-Wire Wire Line
-	14175 8975 14450 8975
-Wire Wire Line
-	13275 9125 13200 9125
-Text GLabel 13200 9125 0    50   Input ~ 0
-XADCGND
-Wire Wire Line
-	12825 8900 12825 8975
-Text GLabel 12825 8900 1    50   Input ~ 0
-AVCC3V3
-Wire Wire Line
-	13275 8975 12825 8975
-$Comp
-L antmicroPMICPowerDistributionSwitchesLoadDrivers:REF3012AIDBZT U?
-U 1 1 643B2A61
-P 13975 8975
-F 0 "U?" H 13725 9190 50  0000 C CNN
-F 1 "REF3012AIDBZT" H 13725 9099 50  0000 C CNN
-F 2 "antmicro-footprints:SOT-23-3" H 14125 9275 50  0001 L BNN
-F 3 "" H 14125 9375 50  0001 L BNN
-	1    13975 8975
-	1    0    0    -1
-$EndComp
-Text GLabel 14425 7650 2    50   Input ~ 0
-AVCC3V3
-Text GLabel 12800 7550 1    50   Input ~ 0
-VCC3V3
-$Comp
-L power:GND #PWR?
-U 1 1 642F2B49
-P 13025 8150
-F 0 "#PWR?" H 13025 7900 50  0001 C CNN
-F 1 "GND" H 13030 7977 50  0000 C CNN
-F 2 "" H 13025 8150 50  0001 C CNN
-F 3 "" H 13025 8150 50  0001 C CNN
-	1    13025 8150
-	1    0    0    -1
-$EndComp
-Wire Wire Line
-	13025 7950 13025 8150
-Wire Wire Line
-	12800 7650 12800 7550
-Wire Wire Line
-	14100 7650 14425 7650
-Connection ~ 14100 7650
-$Comp
-L antmicroCapacitors0402:C_470n_0402 C?
-U 1 1 64284146
-P 14100 7800
-F 0 "C?" H 14215 7845 60  0000 L CNN
-F 1 "C_470n_0402" H 14100 7650 60  0001 C CNN
-F 2 "antmicro-footprints:0402-cap" H 14300 8000 60  0001 L CNN
-F 3 "" H 14100 7800 50  0001 C CNN
-F 4 "TDK" H 14300 8200 60  0001 L CNN "Manufacturer"
-F 5 "C1005X5R1E474M050BB" H 14300 8100 60  0001 L CNN "MPN"
-F 6 "470n" H 14215 7747 50  0000 L CNN "Val"
-	1    14100 7800
-	1    0    0    -1
-$EndComp
-Wire Wire Line
-	13775 7650 14100 7650
-Connection ~ 13775 7650
-Wire Wire Line
-	14100 7950 13775 7950
-Connection ~ 13775 7950
-$Comp
-L antmicroCapacitors0402:C_1u_0402 C?
-U 1 1 64282C33
-P 13775 7800
-F 0 "C?" H 13660 7755 60  0000 R CNN
-F 1 "C_1u_0402" H 13775 7650 60  0001 C CNN
-F 2 "antmicro-footprints:0402-cap" H 13975 8000 60  0001 L CNN
-F 3 "" H 13775 7800 50  0001 C CNN
-F 4 "TDK" H 13975 8200 60  0001 L CNN "Manufacturer"
-F 5 "C1005X6S1A105K050BC" H 13975 8100 60  0001 L CNN "MPN"
-F 6 "1u" H 13660 7853 50  0000 R CNN "Val"
-	1    13775 7800
-	-1   0    0    1
-$EndComp
-Wire Wire Line
-	13500 7650 13775 7650
-Wire Wire Line
-	13400 7650 13500 7650
-Connection ~ 13500 7650
-Wire Wire Line
-	13775 7950 13500 7950
-Wire Wire Line
-	13500 7950 13025 7950
-Connection ~ 13500 7950
-$Comp
-L antmicroCapacitors0402:C_10u_0402 C?
-U 1 1 6427ABFA
-P 13500 7800
-F 0 "C?" H 13385 7755 60  0000 R CNN
-F 1 "C_10u_0402" H 13500 7650 60  0001 C CNN
-F 2 "antmicro-footprints:0402-cap" H 13700 8000 60  0001 L CNN
-F 3 "" H 13500 7800 50  0001 C CNN
-F 4 "MURATA" H 13700 8200 60  0001 L CNN "Manufacturer"
-F 5 "GRM155R60J106ME44D" H 13700 8100 60  0001 L CNN "MPN"
-F 6 "10u" H 13385 7853 50  0000 R CNN "Val"
-	1    13500 7800
-	-1   0    0    1
-$EndComp
-Wire Wire Line
-	13025 7650 12800 7650
-Wire Wire Line
-	13100 7650 13025 7650
-Connection ~ 13025 7650
-Connection ~ 13025 7950
-$Comp
-L antmicroCapacitors0402:C_10u_0402 C?
-U 1 1 642799BF
-P 13025 7800
-F 0 "C?" H 12910 7755 60  0000 R CNN
-F 1 "C_10u_0402" H 13025 7650 60  0001 C CNN
-F 2 "antmicro-footprints:0402-cap" H 13225 8000 60  0001 L CNN
-F 3 "" H 13025 7800 50  0001 C CNN
-F 4 "MURATA" H 13225 8200 60  0001 L CNN "Manufacturer"
-F 5 "GRM155R60J106ME44D" H 13225 8100 60  0001 L CNN "MPN"
-F 6 "10u" H 12910 7853 50  0000 R CNN "Val"
-	1    13025 7800
-	-1   0    0    1
-$EndComp
-$Comp
-L antmicroFixedInductors:10uH L?
-U 1 1 64278577
-P 13250 7650
-F 0 "L?" H 13250 7864 60  0000 C CNN
-F 1 "10uH" H 13250 7758 60  0000 C CNN
-F 2 "antmicro-footprints:0805-res" H 13300 7500 60  0001 C CNN
-F 3 "" H 13305 7680 60  0001 C CNN
-F 4 "TDK" H 13250 7550 50  0001 C CNN "Manufacturer"
-F 5 "MLZ2012N100LT000" H 13200 7600 50  0001 C CNN "MPN"
-	1    13250 7650
-	1    0    0    -1
-$EndComp
-Text GLabel 13200 9500 0    50   Input ~ 0
-XADCGND
-$Comp
-L power:GND #PWR?
-U 1 1 64669A59
-P 13875 9500
-F 0 "#PWR?" H 13875 9250 50  0001 C CNN
-F 1 "GND" V 13880 9372 50  0000 R CNN
-F 2 "" H 13875 9500 50  0001 C CNN
-F 3 "" H 13875 9500 50  0001 C CNN
-	1    13875 9500
-	0    -1   -1   0
-$EndComp
-$Comp
-L antmicroFerriteBeadsandChips:BLM18PG121SN1D FB?
-U 1 1 6466A4B3
-P 13500 9500
-F 0 "FB?" H 13500 9787 60  0000 C CNN
-F 1 "BLM18PG121SN1D" H 13500 9681 60  0000 C CNN
-F 2 "antmicro-footprints:0603-res" H 13700 9700 60  0001 L CNN
-F 3 "https://www.murata.com/en-us/products/productdata/8796738650142/ENFA0003.pdf" H 13700 9800 60  0001 L CNN
-F 4 "BLM18PG121SN1D" H 13700 10000 60  0001 L CNN "MPN"
-F 5 "Murata Electronics North America" H 13700 10600 60  0001 L CNN "Manufacturer"
-	1    13500 9500
-	1    0    0    -1
-$EndComp
-Wire Wire Line
-	13200 9500 13300 9500
-Wire Wire Line
-	13700 9500 13875 9500
+Text Notes 5375 2375 0    118  ~ 0
+VCCAUX decoupling
 $EndSCHEMATC

Commit message: Updated power sequencer
Connections:
- net labels added: VCC1V35_BANK, VCC1V8_BANK, VCC3V3_BANK, VCCAUX, VCCINT
- net labels removed: VCC1V0, VCC1V8, VCCB14, VCCB15, VCCB16, VCCB34, VCCB35
Changed lines of the file:
@@
 	1150 4000 1150 3850
 Connection ~ 1150 4000
-Text GLabel 1150 3850 1    50   Input ~ 0
-VCCB14
 $Comp
 L antmicroCapacitorsmisc:C_47u_1210 C?
@@
 	1150 5100 1150 4950
 Connection ~ 1150 5100
-Text GLabel 1150 4950 1    50   Input ~ 0
-VCCB15
 $Comp
 L antmicroCapacitorsmisc:C_47u_1210 C?
@@
 	1150 6200 1150 6050
 Connection ~ 1150 6200
-Text GLabel 1150 6050 1    50   Input ~ 0
-VCCB16
 $Comp
 L antmicroCapacitorsmisc:C_47u_1210 C?
@@
 	1150 7300 1150 7150
 Connection ~ 1150 7300
-Text GLabel 1150 7150 1    50   Input ~ 0
-VCCB34
 $Comp
 L antmicroCapacitorsmisc:C_47u_1210 C?
@@
 	1150 8400 1150 8250
 Connection ~ 1150 8400
-Text GLabel 1150 8250 1    50   Input ~ 0
-VCCB35
 Wire Wire Line
 	7750 3300 7600 3300
@@
 Wire Wire Line
 	7750 3700 7600 3700
-Text GLabel 7600 3700 0    50   Input ~ 0
-VCC1V8
 Wire Wire Line
 	7750 3600 7600 3600
-Text GLabel 7600 3600 0    50   Input ~ 0
-VCC1V8
 Text GLabel 4650 3800 1    50   Input ~ 0
 XADC1V8
@@
 Text GLabel 4650 4500 3    50   Input ~ 0
 XADCGND
-Text GLabel 7600 2600 1    50   Input ~ 0
-VCC1V8
 $Comp
 L antmicroCapacitorsmisc:C_47u_1210 C?
@@
 	7050 3400 7050 3250
 Connection ~ 7050 3250
-Text GLabel 4650 2600 1    50   Input ~ 0
-VCC1V8
 Wire Wire Line
 	4650 2600 4650 2750
@@
 Wire Wire Line
 	7600 3900 7600 3800
-Text GLabel 7400 3800 0    50   Input ~ 0
-VCC1V0
 Wire Wire Line
 	7600 3800 7400 3800
 Connection ~ 7600 3800
-Text GLabel 9900 2600 1    50   Input ~ 0
-VCC1V0
 $Comp
 L antmicroCapacitorsmisc:C_100u_1210 C?
@@
 Text Notes 5700 4250 0    118  ~ 0
 BRAM decoupling
-Text GLabel 5500 4300 1    50   Input ~ 0
-VCC1V0
 $Comp
 L antmicroCapacitorspol:C_330u_KEMET_D C?
@@
 	11500 4100 11500 3900
 Connection ~ 11500 4100
-Text GLabel 12050 2600 1    50   Input ~ 0
-VCC1V0
-Text GLabel 11500 3900 1    50   Input ~ 0
-VCC1V0
 $Comp
 L antmicroCapacitorspol:C_680u_KEMET_D C?
@@
 Wire Wire Line
 	11000 2800 11000 2600
-Text GLabel 11000 2600 1    50   Input ~ 0
-VCC1V0
 Text Notes 10550 2800 3    50   ~ 0
 populate on \n
@@
 Text Notes 5375 2375 0    118  ~ 0
 VCCAUX decoupling
+Text GLabel 4650 2600 1    50   Input ~ 0
+VCCAUX
+Text GLabel 7600 2600 1    50   Input ~ 0
+VCCAUX
+Text GLabel 7600 3600 0    50   Input ~ 0
+VCCAUX
+Text GLabel 7600 3700 0    50   Input ~ 0
+VCCAUX
+Text GLabel 7400 3800 0    50   Input ~ 0
+VCCINT
+Text GLabel 5500 4300 1    50   Input ~ 0
+VCCINT
+Text GLabel 9900 2600 1    50   Input ~ 0
+VCCINT
+Text GLabel 11000 2600 1    50   Input ~ 0
+VCCINT
+Text GLabel 12050 2600 1    50   Input ~ 0
+VCCINT
+Text GLabel 11500 3900 1    50   Input ~ 0
+VCCINT
+Text GLabel 1150 3850 0    50   Input ~ 0
+VCC1V8_BANK
+Text GLabel 1150 4950 0    50   Input ~ 0
+VCC3V3_BANK
+Text GLabel 1150 6050 0    50   Input ~ 0
+VCC3V3_BANK
+Text GLabel 1150 7150 0    50   Input ~ 0
+VCC1V35_BANK
+Text GLabel 1150 8250 0    50   Input ~ 0
+VCC1V35_BANK
 $EndSCHEMATC

Commit message: Initial component placement added (to be adjusted further)
Parts:
- gave numbers to parts that had none: 88

Commit message: Update after designator unification
Parts:
- renumbered C11 to C100, C12 to C101, C13 to C102, C14 to C103, C15 to C104, C16 to C105, C17 to C106, C18 to C107, C19 to C108, C20 to C109, C21 to C110, C22 to C111, C23 to C112, C24 to C113, C25 to C114, C26 to C115, C27 to C116, C28 to C117, C29 to C118, C30 to C119, C31 to C120, C32 to C121, C33 to C122, C34 to C123, C35 to C124, C36 to C125, C37 to C126, C38 to C127, C39 to C128, C40 to C129, C41 to C130, C42 to C131, C43 to C132, C44 to C133, C45 to C134, C46 to C135, C47 to C136, C48 to C137, C49 to C138, C50 to C139, C51 to C140, C52 to C141, C53 to C142, C54 to C143, C55 to C144, C56 to C145, C57 to C146, C58 to C147, C59 to C148, C60 to C149, C61 to C150, C62 to C151, C63 to C152, C64 to C153, C65 to C154, C66 to C155, C67 to C156, C68 to C157, C69 to C158, C70 to C159, C71 to C160, C72 to C161, C73 to C162, C74 to C163, C75 to C164, C76 to C165, C77 to C166, C78 to C167, C79 to C168, C80 to C169, C81 to C170, C82 to C171, C83 to C172, C84 to C173, C85 to C174, C86 to C175, C87 to C176, C88 to C177, C2 to C91, C3 to C92, C4 to C93, C5 to C94, C6 to C95, C7 to C96, C8 to C97, C9 to C98, C10 to C99, U1 to U14

Commit message: Add local component libraries
Parts:
- C100, C101, C102, C103, C104, C105, C106, C107, C108, C135, C137, C139, C154, C156, C158, C160, C162, C164, C166, C168, C170, C172, C174, C176, C97, C98, C99: footprint antmicro-footprints:0805-cap -> artix-dc-scm-footprints:0805-cap; symbol antmicroCapacitorsmisc:C_4u7_0805 -> artix-dc-scm:C_4u7_0805
- C109, C110, C111, C112, C113, C114, C115, C116, C117, C118, C119, C120, C121, C122, C123, C124, C125, C126, C127, C128, C129, C130, C131, C132, C138, C140, C141, C142, C143, C144, C146, C148, C152, C153, C155, C157, C159, C161, C163, C165, C167, C169, C171, C173, C175, C177: footprint antmicro-footprints:0603-cap -> artix-dc-scm-footprints:0603-cap; symbol antmicroCapacitors0603:C_470n_0603 -> artix-dc-scm:C_470n_0603
- C133, C147, C91, C92, C93, C94, C95, C96: footprint antmicro-footprints:1210-cap -> artix-dc-scm-footprints:1210-cap; symbol antmicroCapacitorsmisc:C_47u_1210 -> artix-dc-scm:C_47u_1210
- C134: footprint antmicro-footprints:0402-cap -> artix-dc-scm-footprints:0402-cap; symbol antmicroCapacitors0402:C_10n_0402 -> artix-dc-scm:C_10n_0402
- C136: footprint antmicro-footprints:0402-cap -> artix-dc-scm-footprints:0402-cap; symbol antmicroCapacitors0402:C_100n_0402 -> artix-dc-scm:C_100n_0402
- C145, C151: footprint antmicro-footprints:1210-cap -> artix-dc-scm-footprints:1210-cap; symbol antmicroCapacitorsmisc:C_100u_1210 -> artix-dc-scm:C_100u_1210
- C149: footprint antmicro-footprints:KEMET_D -> artix-dc-scm-footprints:KEMET_D; symbol antmicroCapacitorspol:C_680u_KEMET_D -> artix-dc-scm:C_680u_KEMET_D
- C150: footprint antmicro-footprints:KEMET_D -> artix-dc-scm-footprints:KEMET_D; symbol antmicroCapacitorspol:C_330u_KEMET_D -> artix-dc-scm:C_330u_KEMET_D
- U14: footprint antmicro-footprints:Xilinx_FGG484 -> artix-dc-scm-footprints:Xilinx_FGG484; symbol antmicroMicrocontrollers:XC7A100T-FGG484 -> artix-dc-scm:XC7A100T-FGG484

Commit message: Component placement done
Parts:
- removed C109, C110, C111, C112, C113, C114, C115, C116, C117, C118, C119, C120, C121, C122, C123, C124, C125, C126, C127, C128, C129, C130, C131, C132, C138, C140, C141, C142, C143, C144, C146, C148, C152, C153, C155, C157, C159, C161, C163, C165, C167, C169, C171, C173, C175, C177: C_470n_0603, artix-dc-scm-footprints:0603-cap, symbol artix-dc-scm:C_470n_0603
- added C109, C110, C111, C112, C113, C114, C115, C116, C117, C118, C119, C120, C121, C122, C123, C124, C125, C126, C127, C128, C129, C130, C131, C132, C138, C140, C141, C142, C143, C144, C146, C148, C152, C153, C155, C157, C159, C161, C163, C165, C167, C169, C171, C173, C175, C177: C_470n_0402, artix-dc-scm-footprints:0402-cap, symbol artix-dc-scm:C_470n_0402
- C100, C101, C102, C103, C104, C105, C106, C107, C108, C135, C137, C139, C154, C156, C158, C160, C162, C164, C166, C168, C170, C172, C174, C176, C97, C98, C99: value C_4u7_0805 -> C_4u7_0603; footprint artix-dc-scm-footprints:0805-cap -> artix-dc-scm-footprints:0603-cap; symbol artix-dc-scm:C_4u7_0805 -> artix-dc-scm:C_4u7_0603; MPN 0805X475K250CT -> 0603X475K250CT
Connections:
- net GND: now also C145.2, C147.2, C109.2, C110.2, C111.2, C112.2, C113.2, C114.2, C115.2, C116.2, C117.2, C118.2, C119.2, C120.2, C121.2, C122.2, C123.2, C124.2, C125.2, C126.2, C127.2, C128.2, C129.2, C130.2, C131.2, C132.2, C138.2, C140.2, C141.2, C142.2, C143.2, C144.2, C146.2, C148.2, C152.2, C153.2, C155.2, C157.2, C159.2, C161.2, C163.2, C165.2, C167.2, C169.2, C171.2, C173.2, C175.2, C177.2
- net VCC1V35_BANK: now also C113.1, C114.1, C119.1, C120.1, C125.1, C126.1, C131.1, C132.1
- net VCC1V8_BANK: now also C110.1, C116.1, C122.1, C128.1
- net VCC3V3_BANK: now also C111.1, C112.1, C117.1, C118.1, C123.1, C124.1, C129.1, C130.1
- net VCCAUX: now also C141.1, C143.1, C144.1, C146.1, C148.1
- net VCCB13: now also C109.1, C115.1, C121.1, C127.1
- net VCCINT: now also C138.1, C140.1, C142.1, C152.1, C153.1, C155.1, C157.1, C159.1, C161.1, C163.1, C165.1, C167.1, C169.1, C171.1, C173.1, C175.1, C177.1
