File: ethernet.sch (KiCad schematic (older format))
At the start: 48 parts

Commit message: Initial component placement added (to be adjusted further)
Parts:
- gave numbers to parts that had none: 48

Commit message: Update after designator unification
Parts:
- renumbered C89 to C1, C98 to C10, C99 to C11, C100 to C12, C101 to C13, C102 to C14, C103 to C15, C104 to C16, C105 to C17, C106 to C18, C107 to C19, C90 to C2, C108 to C20, C109 to C21, C110 to C22, C111 to C23, C112 to C24, C113 to C25, C114 to C26, C91 to C3, C92 to C4, C93 to C5, C94 to C6, C95 to C7, C96 to C8, C97 to C9, J?1 to J1, R11 to R1, R22 to R10, R23 to R11, R24 to R12, R25 to R13, R31 to R14, R32 to R15, R45 to R16, R12 to R2, R13 to R3, R14 to R4, R15 to R5, R16 to R6, R17 to R7, R18 to R8, R19 to R9, U2 to U1

Commit message: Add local component libraries
Parts:
- C1, C10, C18, C22, C6: footprint antmicro-footprints:0402-cap -> artix-dc-scm-footprints:0402-cap; symbol antmicroCapacitors0402:C_4u7_0402 -> artix-dc-scm:C_4u7_0402
- C11, C12, C13, C14, C15, C16, C17, C21, C23, C25, C5, C7, C9: footprint antmicro-footprints:0402-cap -> artix-dc-scm-footprints:0402-cap; symbol antmicroCapacitors0402:C_10n_0402 -> artix-dc-scm:C_10n_0402
- C19, C2, C3, C4, C8: footprint antmicro-footprints:0402-cap -> artix-dc-scm-footprints:0402-cap; symbol antmicroCapacitors0402:C_470n_0402 -> artix-dc-scm:C_470n_0402
- C20, C26: footprint antmicro-footprints:0402-cap -> artix-dc-scm-footprints:0402-cap; symbol antmicroCapacitors0402:C_22p_0402 -> artix-dc-scm:C_22p_0402
- C24: footprint antmicro-footprints:0402-cap -> artix-dc-scm-footprints:0402-cap; symbol antmicroCapacitors0402:C_100n_0402 -> artix-dc-scm:C_100n_0402
- FB1, FB2, FB3: footprint antmicro-footprints:0603-res -> artix-dc-scm-footprints:0603-res; symbol antmicroFerriteBeadsandChips:BLM18PG121SN1D -> artix-dc-scm:BLM18PG121SN1D
- J1: footprint antmicro-footprints:7499111121A -> artix-dc-scm-footprints:7499111121A; symbol antmicroModularConnectorsJacksWithMagnetics:WE-RJ45_7499111121A -> artix-dc-scm:WE-RJ45_7499111121A
- R1, R10, R11, R12, R2, R3, R4, R5, R6, R7, R8, R9: footprint antmicro-footprints:0402-res -> artix-dc-scm-footprints:0402-res; symbol antmicroResistors0402:R_10k2_0402 -> artix-dc-scm:R_10k2_0402
- R13: footprint antmicro-footprints:0402-res -> artix-dc-scm-footprints:0402-res; symbol antmicroResistors0402:R_12k1_0402 -> artix-dc-scm:R_12k1_0402
- R14: footprint antmicro-footprints:0402-res -> artix-dc-scm-footprints:0402-res; symbol antmicroResistors0402:R_1M8_0402 -> artix-dc-scm:R_1M8_0402
- R15, R16: footprint antmicro-footprints:0402-res -> artix-dc-scm-footprints:0402-res; symbol antmicroResistors0402:R_1k_0402 -> artix-dc-scm:R_1k_0402
- U1: footprint antmicro-footprints:QFN-48-Microchip-QFN77-48LD-PL-2 -> artix-dc-scm-footprints:QFN-48-Microchip-QFN77-48LD-PL-2; symbol antmicroInterfaceControllers:KSZ9031RNXCA -> artix-dc-scm:KSZ9031RNXCA
- Y1: footprint antmicro-footprints:KX-7 -> artix-dc-scm-footprints:KX-7; symbol antmicroCrystals:ABM8G-25.000MHZ-18-D2Y-T -> artix-dc-scm:ABM8G-25.000MHZ-18-D2Y-T

Commit message: Replaced PHY
Parts:
- removed C1, C10, C18, C22, C6: C_4u7_0402, artix-dc-scm-footprints:0402-cap, symbol artix-dc-scm:C_4u7_0402
- removed C11, C12, C13, C14, C15, C16, C17, C21, C23, C25, C5, C7, C9: C_10n_0402, artix-dc-scm-footprints:0402-cap, symbol artix-dc-scm:C_10n_0402
- removed C19, C2, C3, C4, C8: C_470n_0402, artix-dc-scm-footprints:0402-cap, symbol artix-dc-scm:C_470n_0402
- removed C20, C26: C_22p_0402, artix-dc-scm-footprints:0402-cap, symbol artix-dc-scm:C_22p_0402
- removed C24: C_100n_0402, artix-dc-scm-footprints:0402-cap, symbol artix-dc-scm:C_100n_0402
- removed FB1, FB2, FB3: BLM18PG121SN1D, artix-dc-scm-footprints:0603-res, symbol artix-dc-scm:BLM18PG121SN1D
- removed J1: WE-RJ45_7499111121A, artix-dc-scm-footprints:7499111121A, symbol artix-dc-scm:WE-RJ45_7499111121A
- removed R1, R10, R11, R12, R2, R3, R4, R5, R6, R7, R8, R9: R_10k2_0402, artix-dc-scm-footprints:0402-res, symbol artix-dc-scm:R_10k2_0402
- removed R13: R_12k1_0402, artix-dc-scm-footprints:0402-res, symbol artix-dc-scm:R_12k1_0402
- removed R14: R_1M8_0402, artix-dc-scm-footprints:0402-res, symbol artix-dc-scm:R_1M8_0402
- removed R15, R16: R_1k_0402, artix-dc-scm-footprints:0402-res, symbol artix-dc-scm:R_1k_0402
- removed U1: KSZ9031RNXCA, artix-dc-scm-footprints:QFN-48-Microchip-QFN77-48LD-PL-2, symbol artix-dc-scm:KSZ9031RNXCA
- removed Y1: ABM8G-25.000MHZ-18-D2Y-T, artix-dc-scm-footprints:KX-7, symbol artix-dc-scm:ABM8G-25.000MHZ-18-D2Y-T
- added C10, C13, C3, C4, C5, C9: C_100n_0402, antmicro-footprints:0402-cap, symbol antmicroCapacitors0402:C_100n_0402
- added C11, C12: C_27p_0402, antmicro-footprints:0402-cap, symbol antmicroCapacitors0402:C_27p_0402
- added C2, C6, C7: C_10u_0603, antmicro-footprints:0603-cap, symbol antmicroCapacitors0603:C_10u_0603
- added C8: C_1u_0402, antmicro-footprints:0402-cap, symbol antmicroCapacitors0402:C_1u_0402
- added FB2: MPZ2012S601AT000, antmicro-footprints:0805-res, symbol antmicroFerriteBeadsandChips:MPZ2012S601AT000
- added J1: 08B0-1X1T-36-F, antmicro-footprints:BEL_08B0-1X1T-36-F, symbol antmicroModularConnectorsJacksWithMagnetics:08B0-1X1T-36-F
- added R10: R_1k5_0402, antmicro-footprints:0402-res, symbol antmicroResistors0402:R_1k5_0402
- added R11: R_0R_0402, antmicro-footprints:0402-res, symbol antmicroResistors0402:R_0R_0402
- added R12, R13: R_220R_0402, antmicro-footprints:0402-res, symbol antmicroResistors0402:R_220R_0402
- added R127, R14, R15, R16: R_49R9_0402, antmicro-footprints:0402-res, symbol antmicroResistors0402:R_49R9_0402
- added R3, R4, R5, R6, R7: R_2k2_0402, antmicro-footprints:0402-res, symbol antmicroResistors0402:R_2k2_0402
- added R8: R_4k87_0402, antmicro-footprints:0402-res, symbol antmicroResistors0402:R_4k87_0402
- added R9: R_10k_0402, antmicro-footprints:0402-res, symbol antmicroResistors0402:R_10k_0402
- added U15: DP83848JSQ_NOPB, antmicro-footprints:DP83848JSQ-NOPB, symbol antmicroInterfaceDriversReceiversTransceivers:DP83848JSQ_NOPB
- added Y2: ABM8G-25.000MHZ-18-D2Y-T, antmicro-footprints:KX-7, symbol antmicroCrystals:ABM8G-25.000MHZ-18-D2Y-T
Connections:
- net labels added: 3V3_SYS, ETH3V3, ETH_COL, ETH_CRS, ETH_REF_CLK, ETH_RSTN, ETH_RXD0, ETH_RXD1, ETH_RXD2, ETH_RXD3, ETH_RXERR, ETH_RX_CLK, ETH_RX_DV, ETH_TXD0, ETH_TXD1, ETH_TXD2, ETH_TXD3, ETH_TX_CLK, ETH_TX_EN, LED_LINK, LED_SPD, PFBOUT, RXN, RXP, TXN, TXP
- net labels removed: AVDDL, AVDDL_PLL, ETH1_N, ETH1_P, ETH2_N, ETH2_P, ETH3_N, ETH3_P, ETH4_N, ETH4_P, ETH_INT_N, ETH_LED1, ETH_LED2, ETH_~RESET, RGMII_REF_CLK, RGMII_RXD0, RGMII_RXD1, RGMII_RXD2, RGMII_RXD3, RGMII_RX_CLK, RGMII_RX_DV, RGMII_TXD0, RGMII_TXD1, RGMII_TXD2, RGMII_TXD3, RGMII_TX_CLK, RGMII_TX_DV, VCC1V2
- wire segments 262 -> 167
Other:
- note added: "Ethernet transceiver"
- note added: "RJ45 Connector"
- note removed: "Pull up resistors"
- note removed: "RJ45 connector"

Commit message: Fixes after review (pin connections)
Parts:
- renumbered U15 to U1
Changed lines of the file:
@@
 P 6175 5250
 AR Path="/5FE270C1/5FEA8148" Ref="U?"  Part="1"
-AR Path="/60570C04/5FEA8148" Ref="U15"  Part="1"
-F 0 "U15" H 5225 6900 50  0000 C CNN
+AR Path="/60570C04/5FEA8148" Ref="U1"  Part="1"
+F 0 "U1" H 5225 6900 50  0000 C CNN
 F 1 "DP83848JSQ_NOPB" H 5525 3550 50  0000 C CNN
 F 2 "antmicro-footprints:DP83848JSQ-NOPB" H 6225 7050 50  0001 L BNN

Commit message: Added USB client chip
Connections:
- net labels removed: 3V3_SYS
Changed lines of the file:
@@
 	3250 4000 3450 4000
 Text GLabel 4400 4450 0    50   Input ~ 0
-3V3_SYS
+VCC3V3
 Wire Wire Line
 	4450 4450 4400 4450

Commit message: New ICs component placement, replaced RJ45
Parts:
- removed J1: 08B0-1X1T-36-F, antmicro-footprints:BEL_08B0-1X1T-36-F, symbol antmicroModularConnectorsJacksWithMagnetics:08B0-1X1T-36-F
- added J?: RJMG1BD3B8K1ANR, CONN_RJMG1BD3B8K1ANR, symbol antmicroModularConnectorsJacksWithMagnetics:RJMG1BD3B8K1ANR
Connections:
- wire segments 167 -> 160
Other:
- moved on the sheet: C13
