File: rot.sch (KiCad schematic (older format))
At the start: 38 parts

Commit message: Added TPM SPI connector
Parts:
- removed J?: 61301021121, antmicro-footprints:61301021121, symbol antmicroRectangularConnectorsHeadersMalePins:61301021121
- removed R? (x4): R_0R_0402, antmicro-footprints:0402-res, symbol antmicroResistors0402:R_0R_0402
- added J?: M20-7830642, antmicro-footprints:PinHeader_6x2_P2.54mm_Vertical, symbol antmicroRectangularConnectorsHeadersFemalePins:M20-7830642
Connections:
- net labels added: GPIO, PIRQ#, PP, RST, SPI0_CLK, SPI0_CS_N, SPI0_MISO, SPI0_MOSI
- net labels removed: 3VSB, CLKRUN, FRAME, ID, LAD0, LAD1, LAD2, LAD3, PCICLK, PCIRST#, PWRDWN, QSPI0_CS1_N, SERIRQ, SUSCLK, VCC3V0
- wire segments 186 -> 169
- no-connect marks 3 -> 0
Other:
- note added: "Pinout for AES-PMOD-TPM20-SLB9670-G"
- note added: "TODO: tie this pins to DC-SCI connector"
- note removed: "This is TPM running on LPC interface, search for some with SPI?"
- note removed: "no pin\n"
Changed lines of the file:
@@
 Text Notes 2525 6300 0    118  ~ 0
 BMC flash
-$Comp
-L antmicroRectangularConnectorsHeadersMalePins:61301021121 J?
-U 1 1 5FEAFE3F
-P 11625 2750
-AR Path="/614223A1/5FEAFE3F" Ref="J?"  Part="1"
-AR Path="/624C566F/5FEAFE3F" Ref="J?"  Part="1"
-F 0 "J?" H 11720 2925 50  0000 C CNN
-F 1 "61301021121" H 11720 2834 50  0000 C CNN
-F 2 "antmicro-footprints:61301021121" V 11425 2000 60  0001 L CNN
-F 3 "" H 11825 3050 60  0001 L CNN
-F 4 "61301021121" H 11825 3250 60  0001 L CNN "MPN"
-F 5 "Wurth Electronics Inc." H 11825 3850 60  0001 L CNN "Manufacturer"
-	1    11625 2750
-	1    0    0    1
-$EndComp
-Wire Wire Line
-	11525 1800 10900 1800
-Text GLabel 10900 1800 0    50   Input ~ 0
-PCICLK
-Text GLabel 10900 1900 0    50   Input ~ 0
-FRAME
-Text GLabel 10900 2100 0    50   Input ~ 0
-LAD3
-Wire Wire Line
-	11525 2200 11425 2200
-Wire Wire Line
-	11425 2200 11425 1650
-Text GLabel 10900 2300 0    50   Input ~ 0
-LAD0
-Text GLabel 10900 2500 0    50   Input ~ 0
-3VSB
-Wire Wire Line
-	11525 1900 10900 1900
-Wire Wire Line
-	11525 2100 10900 2100
-Text GLabel 10900 2000 0    50   Input ~ 0
-PCIRST#
-Wire Wire Line
-	11525 2000 10900 2000
-Wire Wire Line
-	10900 2300 11525 2300
-Wire Wire Line
-	10900 2500 11525 2500
-NoConn ~ 11525 2400
-Wire Wire Line
-	11525 2600 11425 2600
-Wire Wire Line
-	11425 2600 11425 2875
-$Comp
-L power:GND #PWR?
-U 1 1 5FF2F616
-P 11425 2875
-F 0 "#PWR?" H 11425 2625 50  0001 C CNN
-F 1 "GND" H 11430 2702 50  0000 C CNN
-F 2 "" H 11425 2875 50  0001 C CNN
-F 3 "" H 11425 2875 50  0001 C CNN
-	1    11425 2875
-	1    0    0    -1
-$EndComp
-Wire Wire Line
-	11925 1800 12050 1800
-Wire Wire Line
-	12050 1800 12050 2300
-$Comp
-L power:GND #PWR?
-U 1 1 5FF39BDA
-P 12050 2875
-F 0 "#PWR?" H 12050 2625 50  0001 C CNN
-F 1 "GND" H 12055 2702 50  0000 C CNN
-F 2 "" H 12050 2875 50  0001 C CNN
-F 3 "" H 12050 2875 50  0001 C CNN
-	1    12050 2875
-	1    0    0    -1
-$EndComp
-NoConn ~ 11925 1900
-NoConn ~ 11925 2000
-Text GLabel 12550 2100 2    50   Input ~ 0
-LAD2
-Wire Wire Line
-	11925 2100 12550 2100
-Text GLabel 12550 2200 2    50   Input ~ 0
-LAD1
-Wire Wire Line
-	11925 2200 12550 2200
-Wire Wire Line
-	11925 2300 12050 2300
-Connection ~ 12050 2300
-Wire Wire Line
-	12050 2300 12050 2875
-Text GLabel 12550 2400 2    50   Input ~ 0
-ID
-Wire Wire Line
-	11925 2500 12550 2500
-Text GLabel 12550 2500 2    50   Input ~ 0
-SERIRQ
-Text GLabel 12550 2700 2    50   Input ~ 0
-SUSCLK
-Text Notes 11950 1925 0    50   ~ 0
-no pin\n
-Text GLabel 11425 1650 1    50   Input ~ 0
-VCC3V0
-Text GLabel 11025 2700 0    50   Input ~ 0
-PWRDWN
-$Comp
-L antmicroResistors0402:R_0R_0402 R?
-U 1 1 5FF9DBC1
-P 11225 2700
-F 0 "R?" H 11225 2913 60  0000 C CNN
-F 1 "R_0R_0402" H 11225 2550 60  0001 C CNN
-F 2 "antmicro-footprints:0402-res" H 11425 2900 60  0001 L CNN
-F 3 "" H 11225 2700 50  0001 C CNN
-F 4 "PANASONIC" H 11425 3100 60  0001 L CNN "Manufacturer"
-F 5 "ERJ2GE0R00X" H 11425 3000 60  0001 L CNN "MPN"
-F 6 "0R" H 11225 2815 50  0000 C CNN "Val"
-	1    11225 2700
-	1    0    0    -1
-$EndComp
-Wire Wire Line
-	11075 2700 11025 2700
-Wire Wire Line
-	11375 2700 11525 2700
-Text GLabel 12550 2600 2    50   Input ~ 0
-CLKRUN
-$Comp
-L antmicroResistors0402:R_0R_0402 R?
-U 1 1 5FFB3D35
-P 12275 2600
-F 0 "R?" H 12275 2813 60  0000 C CNN
-F 1 "R_0R_0402" H 12275 2450 60  0001 C CNN
-F 2 "antmicro-footprints:0402-res" H 12475 2800 60  0001 L CNN
-F 3 "" H 12275 2600 50  0001 C CNN
-F 4 "PANASONIC" H 12475 3000 60  0001 L CNN "Manufacturer"
-F 5 "ERJ2GE0R00X" H 12475 2900 60  0001 L CNN "MPN"
-F 6 "0R" H 12275 2715 50  0000 C CNN "Val"
-	1    12275 2600
-	1    0    0    -1
-$EndComp
-$Comp
-L antmicroResistors0402:R_0R_0402 R?
-U 1 1 5FFB415C
-P 12275 2700
-F 0 "R?" H 12275 2913 60  0000 C CNN
-F 1 "R_0R_0402" H 12275 2550 60  0001 C CNN
-F 2 "antmicro-footprints:0402-res" H 12475 2900 60  0001 L CNN
-F 3 "" H 12275 2700 50  0001 C CNN
-F 4 "PANASONIC" H 12475 3100 60  0001 L CNN "Manufacturer"
-F 5 "ERJ2GE0R00X" H 12475 3000 60  0001 L CNN "MPN"
-F 6 "0R" H 12275 2815 50  0000 C CNN "Val"
-	1    12275 2700
-	1    0    0    -1
-$EndComp
-Wire Wire Line
-	11925 2700 12125 2700
-Wire Wire Line
-	12425 2700 12550 2700
-Wire Wire Line
-	11925 2600 12125 2600
-Wire Wire Line
-	12425 2600 12550 2600
-$Comp
-L antmicroResistors0402:R_0R_0402 R?
-U 1 1 5FFECBDF
-P 12275 2400
-F 0 "R?" H 12275 2613 60  0000 C CNN
-F 1 "R_0R_0402" H 12275 2250 60  0001 C CNN
-F 2 "antmicro-footprints:0402-res" H 12475 2600 60  0001 L CNN
-F 3 "" H 12275 2400 50  0001 C CNN
-F 4 "PANASONIC" H 12475 2800 60  0001 L CNN "Manufacturer"
-F 5 "ERJ2GE0R00X" H 12475 2700 60  0001 L CNN "MPN"
-F 6 "0R" H 12275 2515 50  0000 C CNN "Val"
-	1    12275 2400
-	1    0    0    -1
-$EndComp
-Wire Wire Line
-	12550 2400 12425 2400
-Wire Wire Line
-	12125 2400 11925 2400
-Text Notes 10975 1075 0    118  ~ 0
+Text Notes 10900 1500 0    118  ~ 0
 TPM connector
 Text Notes 1650 6400 0    50   ~ 0
@@
 Text Notes 1475 1475 0    50   ~ 0
 One or typically two flash devices used to contain the BIOS firmware image
-Text Notes 11050 3225 0    50   ~ 0
-This is TPM running on LPC interface, search for some with SPI?
 Text GLabel 8250 4900 0    50   Input ~ 0
 SPI_ROT_CLK
@@
 Text GLabel 9700 5300 2    50   Input ~ 0
 QSPI0_D3
-Text GLabel 12825 3375 2    50   Input ~ 0
-QSPI0_CS1_N
 Wire Wire Line
 	8250 5300 8750 5300
@@
 Text Notes 10525 5325 1    50   ~ 0
 QSPI to HPM
-Text GLabel 12825 3475 2    50   Input ~ 0
-QSPI0_CLK
-Text GLabel 12825 3575 2    50   Input ~ 0
-QSPI0_D0
-Text GLabel 12825 3675 2    50   Input ~ 0
-QSPI0_D1
-Text GLabel 12825 3775 2    50   Input ~ 0
-QSPI0_D2
-Text GLabel 12825 3875 2    50   Input ~ 0
-QSPI0_D3
 Text GLabel 8250 6800 0    50   Input ~ 0
 ROT_RDY
 Wire Wire Line
 	8750 6800 8250 6800
+$Comp
+L antmicroRectangularConnectorsHeadersFemalePins:M20-7830642 J?
+U 1 1 5FD63CCC
+P 11725 2200
+F 0 "J?" H 11725 2647 60  0000 C CNN
+F 1 "M20-7830642" H 11725 2541 60  0000 C CNN
+F 2 "antmicro-footprints:PinHeader_6x2_P2.54mm_Vertical" H 11925 2400 60  0001 L CNN
+F 3 "" H 11925 2500 60  0001 L CNN
+F 4 "M20-7830642" H 11925 2700 60  0001 L CNN "MPN"
+F 5 "Molex" H 11925 2800 60  0001 L CNN "Manufacturer"
+	1    11725 2200
+	1    0    0    -1
+$EndComp
+Text GLabel 10900 1950 1    50   Input ~ 0
+VCC3V3
+Text GLabel 11525 2000 0    50   Input ~ 0
+SPI0_CS_N
+Text GLabel 11525 2100 0    50   Input ~ 0
+SPI0_MOSI
+Text GLabel 11525 2200 0    50   Input ~ 0
+SPI0_MISO
+Text GLabel 11525 2300 0    50   Input ~ 0
+SPI0_CLK
+Text GLabel 11925 2000 2    50   Input ~ 0
+PIRQ#
+Text GLabel 11925 2100 2    50   Input ~ 0
+RST
+Text GLabel 11925 2200 2    50   Input ~ 0
+GPIO
+Text GLabel 11925 2300 2    50   Input ~ 0
+PP
+Text GLabel 12375 1950 1    50   Input ~ 0
+VCC3V3
+Wire Wire Line
+	11525 2500 10900 2500
+Wire Wire Line
+	10900 2500 10900 1950
+Wire Wire Line
+	11925 2500 12375 2500
+Wire Wire Line
+	12375 2500 12375 1950
+Wire Wire Line
+	11525 2400 11400 2400
+Wire Wire Line
+	11400 2400 11400 2650
+Wire Wire Line
+	11925 2400 12050 2400
+Wire Wire Line
+	12050 2400 12050 2650
+$Comp
+L power:GND #PWR?
+U 1 1 5FD82134
+P 11400 2650
+AR Path="/5FC6B687/5FD82134" Ref="#PWR?"  Part="1"
+AR Path="/624C566F/5FD82134" Ref="#PWR?"  Part="1"
+F 0 "#PWR?" H 11400 2400 50  0001 C CNN
+F 1 "GND" H 11405 2477 50  0000 C CNN
+F 2 "" H 11400 2650 50  0001 C CNN
+F 3 "" H 11400 2650 50  0001 C CNN
+	1    11400 2650
+	1    0    0    -1
+$EndComp
+$Comp
+L power:GND #PWR?
+U 1 1 5FD8331F
+P 12050 2650
+AR Path="/5FC6B687/5FD8331F" Ref="#PWR?"  Part="1"
+AR Path="/624C566F/5FD8331F" Ref="#PWR?"  Part="1"
+F 0 "#PWR?" H 12050 2400 50  0001 C CNN
+F 1 "GND" H 12055 2477 50  0000 C CNN
+F 2 "" H 12050 2650 50  0001 C CNN
+F 3 "" H 12050 2650 50  0001 C CNN
+	1    12050 2650
+	1    0    0    -1
+$EndComp
+Text Notes 12175 2675 0    50   ~ 0
+Pinout for AES-PMOD-TPM20-SLB9670-G
+Text Notes 12325 2425 1    50   ~ 0
+TODO: tie this pins to DC-SCI connector
 $EndSCHEMATC

Commit message: Initial component placement added (to be adjusted further)
Parts:
- gave numbers to parts that had none: 34

Commit message: Update after designator unification
Parts:
- U2: renamed from U16; footprint antmicro-footprints:SOIC-8_W5.6mm -> antmicro-footprints:W25Q32JVSSIQ
- U3: renamed from U17; footprint antmicro-footprints:SOIC-8_W5.6mm -> antmicro-footprints:W25Q32JVSSIQ
- U4: renamed from U18; footprint antmicro-footprints:SOIC-8_W5.6mm -> antmicro-footprints:W25Q32JVSSIQ
- U5: renamed from U19; footprint antmicro-footprints:SOIC-8_W5.6mm -> antmicro-footprints:W25Q32JVSSIQ
- renumbered C167 to C35, C168 to C36, C169 to C37, C170 to C38, J10 to J3, J11 to J4, R74 to R21, R75 to R22, R76 to R23, R77 to R24, R78 to R25, R79 to R26, R80 to R27, R81 to R28, R82 to R29, R83 to R30, R84 to R31, R85 to R32, R86 to R33, R87 to R34, R88 to R35, R89 to R36, R90 to R37, R91 to R38, R92 to R39, R93 to R40, R94 to R41, R95 to R42, R96 to R43, R97 to R44

Commit message: Add local component libraries
Parts:
- C35, C36, C37, C38: footprint antmicro-footprints:0402-cap -> artix-dc-scm-footprints:0402-cap; symbol antmicroCapacitors0402:C_470n_0402 -> artix-dc-scm:C_470n_0402
- J3: footprint antmicro-footprints:543630489 -> artix-dc-scm-footprints:543630489; symbol antmicroB2bConnectors:543630489 -> artix-dc-scm:543630489
- J4: footprint antmicro-footprints:PinHeader_6x2_P2.54mm_Vertical -> artix-dc-scm-footprints:PinHeader_6x2_P2.54mm_Vertical; symbol antmicroRectangularConnectorsHeadersFemalePins:M20-7830642 -> artix-dc-scm:M20-7830642
- R21, R22, R23, R24: footprint antmicro-footprints:0402-res -> artix-dc-scm-footprints:0402-res; symbol antmicroResistors0402:R_4k7_0402 -> artix-dc-scm:R_4k7_0402
- R25, R26, R27, R28: footprint antmicro-footprints:0402-res -> artix-dc-scm-footprints:0402-res; symbol antmicroResistors0402:R_1k_0402 -> artix-dc-scm:R_1k_0402
- R29, R30, R31, R32, R33, R34, R35, R36, R37, R38, R39, R40, R41, R42, R43, R44: footprint antmicro-footprints:0402-res -> artix-dc-scm-footprints:0402-res; symbol antmicroResistors0402:R_10k_0402 -> artix-dc-scm:R_10k_0402
- U2, U3, U4, U5: footprint antmicro-footprints:W25Q32JVSSIQ -> artix-dc-scm-footprints:W25Q32JVSSIQ; symbol antmicroMemory:W25Q32JVSSIQ_TR -> artix-dc-scm:W25Q32JVSSIQ_TR
