File: pcie-conn.sch (KiCad schematic (older format))
At the start: 14 parts

Commit message: Initial component placement added (to be adjusted further)
Parts:
- gave numbers to parts that had none: 14
Changed lines of the file:
@@
 	6250 2750 6450 2750
 $Comp
-L antmicroCapacitors0402:C_100n_0402 C?
+L antmicroCapacitors0402:C_100n_0402 C171
 U 1 1 5FD1CF34
 P 6600 2750
-F 0 "C?" V 6342 2750 60  0000 C CNN
+F 0 "C171" V 6342 2750 60  0000 C CNN
 F 1 "C_100n_0402" H 6600 2600 60  0001 C CNN
 F 2 "antmicro-footprints:0402-cap" H 6800 2950 60  0001 L CNN
@@
 $EndComp
 $Comp
-L antmicroCapacitors0402:C_100n_0402 C?
+L antmicroCapacitors0402:C_100n_0402 C173
 U 1 1 5FD1DAE4
 P 6875 2850
-F 0 "C?" V 6617 2850 60  0000 C CNN
+F 0 "C173" V 6617 2850 60  0000 C CNN
 F 1 "C_100n_0402" H 6875 2700 60  0001 C CNN
 F 2 "antmicro-footprints:0402-cap" H 7075 3050 60  0001 L CNN
@@
 	6250 3350 6450 3350
 $Comp
-L antmicroCapacitors0402:C_100n_0402 C?
+L antmicroCapacitors0402:C_100n_0402 C172
 U 1 1 5FD279F6
 P 6600 3350
-F 0 "C?" V 6342 3350 60  0000 C CNN
+F 0 "C172" V 6342 3350 60  0000 C CNN
 F 1 "C_100n_0402" H 6600 3200 60  0001 C CNN
 F 2 "antmicro-footprints:0402-cap" H 6800 3550 60  0001 L CNN
@@
 $EndComp
 $Comp
-L antmicroCapacitors0402:C_100n_0402 C?
+L antmicroCapacitors0402:C_100n_0402 C174
 U 1 1 5FD279FF
 P 6875 3450
-F 0 "C?" V 6617 3450 60  0000 C CNN
+F 0 "C174" V 6617 3450 60  0000 C CNN
 F 1 "C_100n_0402" H 6875 3300 60  0001 C CNN
 F 2 "antmicro-footprints:0402-cap" H 7075 3650 60  0001 L CNN
@@
 	7025 3450 7350 3450
 $Comp
-L antmicroPciConnectors:1-2199230-6 J?
+L antmicroPciConnectors:1-2199230-6 J12
 U 1 1 5FD380A4
 P 5450 3900
-F 0 "J?" H 5450 6565 60  0000 C CNN
+F 0 "J12" H 5450 6565 60  0000 C CNN
 F 1 "1-2199230-6" H 5300 2200 60  0001 C CNN
 F 2 "antmicro-footprints:1-2199230-6" H 5300 2200 60  0001 C CNN
@@
 	3675 2750 4050 2750
 $Comp
-L antmicroResistors0402:R_10k_0402 R?
+L antmicroResistors0402:R_10k_0402 R98
 U 1 1 5FD6D5E7
 P 3825 2125
-F 0 "R?" V 3780 2195 60  0000 L CNN
+F 0 "R98" V 3780 2195 60  0000 L CNN
 F 1 "R_10k_0402" H 3825 1975 60  0001 C CNN
 F 2 "antmicro-footprints:0402-res" H 4025 2325 60  0001 L CNN
@@
 $EndComp
 $Comp
-L antmicroResistors0402:R_10k_0402 R?
+L antmicroResistors0402:R_10k_0402 R100
 U 1 1 5FD6DA61
 P 4050 2125
-F 0 "R?" V 4005 2195 60  0000 L CNN
+F 0 "R100" V 4005 2195 60  0000 L CNN
 F 1 "R_10k_0402" H 4050 1975 60  0001 C CNN
 F 2 "antmicro-footprints:0402-res" H 4250 2325 60  0001 L CNN
@@
 $EndComp
 $Comp
-L antmicroResistors0402:R_10k_0402 R?
+L antmicroResistors0402:R_10k_0402 R101
 U 1 1 5FD7820E
 P 4275 2125
-F 0 "R?" V 4230 2195 60  0000 L CNN
+F 0 "R101" V 4230 2195 60  0000 L CNN
 F 1 "R_10k_0402" H 4275 1975 60  0001 C CNN
 F 2 "antmicro-footprints:0402-res" H 4475 2325 60  0001 L CNN
@@
 	4275 1500 4275 1975
 $Comp
-L antmicroLEDIndicationDiscrete:KP-1608CGCK D?
+L antmicroLEDIndicationDiscrete:KP-1608CGCK D10
 U 1 1 5FD7D8E8
 P 4250 4750
-F 0 "D?" H 4200 5087 60  0000 C CNN
+F 0 "D10" H 4200 5087 60  0000 C CNN
 F 1 "KP-1608CGCK" H 4200 4981 60  0000 C CNN
 F 2 "antmicro-footprints:LED_0603" H 4450 4950 60  0001 L CNN
@@
 	4350 4750 4650 4750
 $Comp
-L antmicroResistors0402:R_330R_0402 R?
+L antmicroResistors0402:R_330R_0402 R99
 U 1 1 5FD7EE61
 P 3850 4375
-F 0 "R?" V 3805 4445 60  0000 L CNN
+F 0 "R99" V 3805 4445 60  0000 L CNN
 F 1 "R_330R_0402" H 3850 4225 60  0001 C CNN
 F 2 "antmicro-footprints:0402-res" H 4050 4575 60  0001 L CNN
@@
 	4550 5350 4550 5675
 $Comp
-L power:GND #PWR?
+L power:GND #PWR095
 U 1 1 5FDC4FA1
 P 4550 5675
-F 0 "#PWR?" H 4550 5425 50  0001 C CNN
+F 0 "#PWR095" H 4550 5425 50  0001 C CNN
 F 1 "GND" H 4555 5502 50  0000 C CNN
 F 2 "" H 4550 5675 50  0001 C CNN
@@
 $EndComp
 $Comp
-L power:GND #PWR?
+L power:GND #PWR096
 U 1 1 5FDC53F7
 P 6325 5675
-F 0 "#PWR?" H 6325 5425 50  0001 C CNN
+F 0 "#PWR096" H 6325 5425 50  0001 C CNN
 F 1 "GND" H 6330 5502 50  0000 C CNN
 F 2 "" H 6325 5675 50  0001 C CNN
@@
 $EndComp
 $Comp
-L antmicroCapacitors0402:C_10u_0402 C?
+L antmicroCapacitors0402:C_10u_0402 C175
 U 1 1 5FDCA87A
 P 7100 5000
-F 0 "C?" H 7215 5045 60  0000 L CNN
+F 0 "C175" H 7215 5045 60  0000 L CNN
 F 1 "C_10u_0402" H 7100 4850 60  0001 C CNN
 F 2 "antmicro-footprints:0402-cap" H 7300 5200 60  0001 L CNN
@@
 $EndComp
 $Comp
-L antmicroCapacitors0402:C_10u_0402 C?
+L antmicroCapacitors0402:C_10u_0402 C176
 U 1 1 5FDCB4B9
 P 7450 5000
-F 0 "C?" H 7565 5045 60  0000 L CNN
+F 0 "C176" H 7565 5045 60  0000 L CNN
 F 1 "C_10u_0402" H 7450 4850 60  0001 C CNN
 F 2 "antmicro-footprints:0402-cap" H 7650 5200 60  0001 L CNN
@@
 $EndComp
 $Comp
-L antmicroCapacitors0402:C_10u_0402 C?
+L antmicroCapacitors0402:C_10u_0402 C177
 U 1 1 5FDCB85E
 P 7800 5000
-F 0 "C?" H 7915 5045 60  0000 L CNN
+F 0 "C177" H 7915 5045 60  0000 L CNN
 F 1 "C_10u_0402" H 7800 4850 60  0001 C CNN
 F 2 "antmicro-footprints:0402-cap" H 8000 5200 60  0001 L CNN
@@
 $EndComp
 $Comp
-L antmicroCapacitors0402:C_10u_0402 C?
+L antmicroCapacitors0402:C_10u_0402 C178
 U 1 1 5FDCBB8F
 P 8150 5000
-F 0 "C?" H 8265 5045 60  0000 L CNN
+F 0 "C178" H 8265 5045 60  0000 L CNN
 F 1 "C_10u_0402" H 8150 4850 60  0001 C CNN
 F 2 "antmicro-footprints:0402-cap" H 8350 5200 60  0001 L CNN
@@
 $EndComp
 $Comp
-L power:GND #PWR?
+L power:GND #PWR097
 U 1 1 5FDD1861
 P 7100 5150
-F 0 "#PWR?" H 7100 4900 50  0001 C CNN
+F 0 "#PWR097" H 7100 4900 50  0001 C CNN
 F 1 "GND" H 7105 4977 50  0000 C CNN
 F 2 "" H 7100 5150 50  0001 C CNN
@@
 $EndComp
 $Comp
-L power:GND #PWR?
+L power:GND #PWR098
 U 1 1 5FDD1B5A
 P 7450 5150
-F 0 "#PWR?" H 7450 4900 50  0001 C CNN
+F 0 "#PWR098" H 7450 4900 50  0001 C CNN
 F 1 "GND" H 7455 4977 50  0000 C CNN
 F 2 "" H 7450 5150 50  0001 C CNN
@@
 $EndComp
 $Comp
-L power:GND #PWR?
+L power:GND #PWR099
 U 1 1 5FDD1D85
 P 7800 5150
-F 0 "#PWR?" H 7800 4900 50  0001 C CNN
+F 0 "#PWR099" H 7800 4900 50  0001 C CNN
 F 1 "GND" H 7805 4977 50  0000 C CNN
 F 2 "" H 7800 5150 50  0001 C CNN
@@
 $EndComp
 $Comp
-L power:GND #PWR?
+L power:GND #PWR0100
 U 1 1 5FDD200B
 P 8150 5150
-F 0 "#PWR?" H 8150 4900 50  0001 C CNN
+F 0 "#PWR0100" H 8150 4900 50  0001 C CNN
 F 1 "GND" H 8155 4977 50  0000 C CNN
 F 2 "" H 8150 5150 50  0001 C CNN

Commit message: Update after designator unification
Parts:
- renumbered C171 to C27, C172 to C28, C173 to C29, C174 to C30, C175 to C31, C176 to C32, C177 to C33, C178 to C34, D10 to D1, J12 to J2, R98 to R17, R99 to R18, R100 to R19, R101 to R20
Changed lines of the file:
@@
 $Descr A4 11693 8268
 encoding utf-8
-Sheet 10 10
+Sheet 3 10
 Title ""
 Date ""
@@
 	6250 2750 6450 2750
 $Comp
-L antmicroCapacitors0402:C_100n_0402 C171
+L antmicroCapacitors0402:C_100n_0402 C27
 U 1 1 5FD1CF34
 P 6600 2750
-F 0 "C171" V 6342 2750 60  0000 C CNN
+F 0 "C27" V 6342 2750 60  0000 C CNN
 F 1 "C_100n_0402" H 6600 2600 60  0001 C CNN
 F 2 "antmicro-footprints:0402-cap" H 6800 2950 60  0001 L CNN
@@
 $EndComp
 $Comp
-L antmicroCapacitors0402:C_100n_0402 C173
+L antmicroCapacitors0402:C_100n_0402 C29
 U 1 1 5FD1DAE4
 P 6875 2850
-F 0 "C173" V 6617 2850 60  0000 C CNN
+F 0 "C29" V 6617 2850 60  0000 C CNN
 F 1 "C_100n_0402" H 6875 2700 60  0001 C CNN
 F 2 "antmicro-footprints:0402-cap" H 7075 3050 60  0001 L CNN
@@
 	6250 3350 6450 3350
 $Comp
-L antmicroCapacitors0402:C_100n_0402 C172
+L antmicroCapacitors0402:C_100n_0402 C28
 U 1 1 5FD279F6
 P 6600 3350
-F 0 "C172" V 6342 3350 60  0000 C CNN
+F 0 "C28" V 6342 3350 60  0000 C CNN
 F 1 "C_100n_0402" H 6600 3200 60  0001 C CNN
 F 2 "antmicro-footprints:0402-cap" H 6800 3550 60  0001 L CNN
@@
 $EndComp
 $Comp
-L antmicroCapacitors0402:C_100n_0402 C174
+L antmicroCapacitors0402:C_100n_0402 C30
 U 1 1 5FD279FF
 P 6875 3450
-F 0 "C174" V 6617 3450 60  0000 C CNN
+F 0 "C30" V 6617 3450 60  0000 C CNN
 F 1 "C_100n_0402" H 6875 3300 60  0001 C CNN
 F 2 "antmicro-footprints:0402-cap" H 7075 3650 60  0001 L CNN
@@
 	7025 3450 7350 3450
 $Comp
-L antmicroPciConnectors:1-2199230-6 J12
+L antmicroPciConnectors:1-2199230-6 J2
 U 1 1 5FD380A4
 P 5450 3900
-F 0 "J12" H 5450 6565 60  0000 C CNN
+F 0 "J2" H 5450 6565 60  0000 C CNN
 F 1 "1-2199230-6" H 5300 2200 60  0001 C CNN
 F 2 "antmicro-footprints:1-2199230-6" H 5300 2200 60  0001 C CNN
@@
 	3675 2750 4050 2750
 $Comp
-L antmicroResistors0402:R_10k_0402 R98
+L antmicroResistors0402:R_10k_0402 R17
 U 1 1 5FD6D5E7
 P 3825 2125
-F 0 "R98" V 3780 2195 60  0000 L CNN
+F 0 "R17" V 3780 2195 60  0000 L CNN
 F 1 "R_10k_0402" H 3825 1975 60  0001 C CNN
 F 2 "antmicro-footprints:0402-res" H 4025 2325 60  0001 L CNN
@@
 $EndComp
 $Comp
-L antmicroResistors0402:R_10k_0402 R100
+L antmicroResistors0402:R_10k_0402 R19
 U 1 1 5FD6DA61
 P 4050 2125
-F 0 "R100" V 4005 2195 60  0000 L CNN
+F 0 "R19" V 4005 2195 60  0000 L CNN
 F 1 "R_10k_0402" H 4050 1975 60  0001 C CNN
 F 2 "antmicro-footprints:0402-res" H 4250 2325 60  0001 L CNN
@@
 $EndComp
 $Comp
-L antmicroResistors0402:R_10k_0402 R101
+L antmicroResistors0402:R_10k_0402 R20
 U 1 1 5FD7820E
 P 4275 2125
-F 0 "R101" V 4230 2195 60  0000 L CNN
+F 0 "R20" V 4230 2195 60  0000 L CNN
 F 1 "R_10k_0402" H 4275 1975 60  0001 C CNN
 F 2 "antmicro-footprints:0402-res" H 4475 2325 60  0001 L CNN
@@
 	4275 1500 4275 1975
 $Comp
-L antmicroLEDIndicationDiscrete:KP-1608CGCK D10
+L antmicroLEDIndicationDiscrete:KP-1608CGCK D1
 U 1 1 5FD7D8E8
 P 4250 4750
-F 0 "D10" H 4200 5087 60  0000 C CNN
+F 0 "D1" H 4200 5087 60  0000 C CNN
 F 1 "KP-1608CGCK" H 4200 4981 60  0000 C CNN
 F 2 "antmicro-footprints:LED_0603" H 4450 4950 60  0001 L CNN
@@
 	4350 4750 4650 4750
 $Comp
-L antmicroResistors0402:R_330R_0402 R99
+L antmicroResistors0402:R_330R_0402 R18
 U 1 1 5FD7EE61
 P 3850 4375
-F 0 "R99" V 3805 4445 60  0000 L CNN
+F 0 "R18" V 3805 4445 60  0000 L CNN
 F 1 "R_330R_0402" H 3850 4225 60  0001 C CNN
 F 2 "antmicro-footprints:0402-res" H 4050 4575 60  0001 L CNN
@@
 	4550 5350 4550 5675
 $Comp
-L power:GND #PWR095
+L power:GND #PWR010
 U 1 1 5FDC4FA1
 P 4550 5675
-F 0 "#PWR095" H 4550 5425 50  0001 C CNN
+F 0 "#PWR010" H 4550 5425 50  0001 C CNN
 F 1 "GND" H 4555 5502 50  0000 C CNN
 F 2 "" H 4550 5675 50  0001 C CNN
@@
 $EndComp
 $Comp
-L power:GND #PWR096
+L power:GND #PWR011
 U 1 1 5FDC53F7
 P 6325 5675
-F 0 "#PWR096" H 6325 5425 50  0001 C CNN
+F 0 "#PWR011" H 6325 5425 50  0001 C CNN
 F 1 "GND" H 6330 5502 50  0000 C CNN
 F 2 "" H 6325 5675 50  0001 C CNN
@@
 $EndComp
 $Comp
-L antmicroCapacitors0402:C_10u_0402 C175
+L antmicroCapacitors0402:C_10u_0402 C31
 U 1 1 5FDCA87A
 P 7100 5000
-F 0 "C175" H 7215 5045 60  0000 L CNN
+F 0 "C31" H 7215 5045 60  0000 L CNN
 F 1 "C_10u_0402" H 7100 4850 60  0001 C CNN
 F 2 "antmicro-footprints:0402-cap" H 7300 5200 60  0001 L CNN
@@
 $EndComp
 $Comp
-L antmicroCapacitors0402:C_10u_0402 C176
+L antmicroCapacitors0402:C_10u_0402 C32
 U 1 1 5FDCB4B9
 P 7450 5000
-F 0 "C176" H 7565 5045 60  0000 L CNN
+F 0 "C32" H 7565 5045 60  0000 L CNN
 F 1 "C_10u_0402" H 7450 4850 60  0001 C CNN
 F 2 "antmicro-footprints:0402-cap" H 7650 5200 60  0001 L CNN
@@
 $EndComp
 $Comp
-L antmicroCapacitors0402:C_10u_0402 C177
+L antmicroCapacitors0402:C_10u_0402 C33
 U 1 1 5FDCB85E
 P 7800 5000
-F 0 "C177" H 7915 5045 60  0000 L CNN
+F 0 "C33" H 7915 5045 60  0000 L CNN
 F 1 "C_10u_0402" H 7800 4850 60  0001 C CNN
 F 2 "antmicro-footprints:0402-cap" H 8000 5200 60  0001 L CNN
@@
 $EndComp
 $Comp
-L antmicroCapacitors0402:C_10u_0402 C178
+L antmicroCapacitors0402:C_10u_0402 C34
 U 1 1 5FDCBB8F
 P 8150 5000
-F 0 "C178" H 8265 5045 60  0000 L CNN
+F 0 "C34" H 8265 5045 60  0000 L CNN
 F 1 "C_10u_0402" H 8150 4850 60  0001 C CNN
 F 2 "antmicro-footprints:0402-cap" H 8350 5200 60  0001 L CNN
@@
 $EndComp
 $Comp
-L power:GND #PWR097
+L power:GND #PWR012
 U 1 1 5FDD1861
 P 7100 5150
-F 0 "#PWR097" H 7100 4900 50  0001 C CNN
+F 0 "#PWR012" H 7100 4900 50  0001 C CNN
 F 1 "GND" H 7105 4977 50  0000 C CNN
 F 2 "" H 7100 5150 50  0001 C CNN
@@
 $EndComp
 $Comp
-L power:GND #PWR098
+L power:GND #PWR013
 U 1 1 5FDD1B5A
 P 7450 5150
-F 0 "#PWR098" H 7450 4900 50  0001 C CNN
+F 0 "#PWR013" H 7450 4900 50  0001 C CNN
 F 1 "GND" H 7455 4977 50  0000 C CNN
 F 2 "" H 7450 5150 50  0001 C CNN
@@
 $EndComp
 $Comp
-L power:GND #PWR099
+L power:GND #PWR014
 U 1 1 5FDD1D85
 P 7800 5150
-F 0 "#PWR099" H 7800 4900 50  0001 C CNN
+F 0 "#PWR014" H 7800 4900 50  0001 C CNN
 F 1 "GND" H 7805 4977 50  0000 C CNN
 F 2 "" H 7800 5150 50  0001 C CNN
@@
 $EndComp
 $Comp
-L power:GND #PWR0100
+L power:GND #PWR015
 U 1 1 5FDD200B
 P 8150 5150
-F 0 "#PWR0100" H 8150 4900 50  0001 C CNN
+F 0 "#PWR015" H 8150 4900 50  0001 C CNN
 F 1 "GND" H 8155 4977 50  0000 C CNN
 F 2 "" H 8150 5150 50  0001 C CNN

Commit message: Changed PCIe connection
Parts:
- added C179, C180, C181, C182: C_100n_0402, antmicro-footprints:0402-cap, symbol antmicroCapacitors0402:C_100n_0402
Connections:
- net labels added: PCIE_HPM_RXN[1], PCIE_HPM_RXN[2], PCIE_HPM_RXN[3], PCIE_HPM_RXP[1], PCIE_HPM_RXP[2], PCIE_HPM_RXP[3], PCIE_HPM_TXN[1], PCIE_HPM_TXN[2], PCIE_HPM_TXN[3], PCIE_HPM_TXP[1], PCIE_HPM_TXP[2], PCIE_HPM_TXP[3]
- wire segments 82 -> 94
- no-connect marks 29 -> 21
Other:
- note removed: "Trellis reference leftovers from PCIe x2"

Commit message: Add local component libraries
Parts:
- C179, C180, C181, C182, C27, C28, C29, C30: footprint antmicro-footprints:0402-cap -> artix-dc-scm-footprints:0402-cap; symbol antmicroCapacitors0402:C_100n_0402 -> artix-dc-scm:C_100n_0402
- C31, C32, C33, C34: footprint antmicro-footprints:0402-cap -> artix-dc-scm-footprints:0402-cap; symbol antmicroCapacitors0402:C_10u_0402 -> artix-dc-scm:C_10u_0402
- D1: footprint antmicro-footprints:LED_0603 -> artix-dc-scm-footprints:LED_0603; symbol antmicroLEDIndicationDiscrete:KP-1608CGCK -> artix-dc-scm:KP-1608CGCK
- J2: footprint antmicro-footprints:1-2199230-6 -> artix-dc-scm-footprints:1-2199230-6; symbol antmicroPciConnectors:1-2199230-6 -> artix-dc-scm:1-2199230-6
- R17, R19, R20: footprint antmicro-footprints:0402-res -> artix-dc-scm-footprints:0402-res; symbol antmicroResistors0402:R_10k_0402 -> artix-dc-scm:R_10k_0402
- R18: footprint antmicro-footprints:0402-res -> artix-dc-scm-footprints:0402-res; symbol antmicroResistors0402:R_330R_0402 -> artix-dc-scm:R_330R_0402
Changed lines of the file:
@@
 	6250 2750 6450 2750
 $Comp
-L antmicroCapacitors0402:C_100n_0402 C27
+L artix-dc-scm:C_100n_0402 C27
 U 1 1 5FD1CF34
 P 6600 2750
 F 0 "C27" V 6342 2750 60  0000 C CNN
 F 1 "C_100n_0402" H 6600 2600 60  0001 C CNN
-F 2 "antmicro-footprints:0402-cap" H 6800 2950 60  0001 L CNN
+F 2 "artix-dc-scm-footprints:0402-cap" H 6800 2950 60  0001 L CNN
 F 3 "" H 6600 2750 50  0001 C CNN
 F 4 "Walsin" H 6800 3150 60  0001 L CNN "Manufacturer"
@@
 $EndComp
 $Comp
-L antmicroCapacitors0402:C_100n_0402 C29
+L artix-dc-scm:C_100n_0402 C29
 U 1 1 5FD1DAE4
 P 6875 2850
 F 0 "C29" V 6617 2850 60  0000 C CNN
 F 1 "C_100n_0402" H 6875 2700 60  0001 C CNN
-F 2 "antmicro-footprints:0402-cap" H 7075 3050 60  0001 L CNN
+F 2 "artix-dc-scm-footprints:0402-cap" H 7075 3050 60  0001 L CNN
 F 3 "" H 6875 2850 50  0001 C CNN
 F 4 "Walsin" H 7075 3250 60  0001 L CNN "Manufacturer"
@@
 	6250 3350 6450 3350
 $Comp
-L antmicroCapacitors0402:C_100n_0402 C28
+L artix-dc-scm:C_100n_0402 C28
 U 1 1 5FD279F6
 P 6600 3350
 F 0 "C28" V 6342 3350 60  0000 C CNN
 F 1 "C_100n_0402" H 6600 3200 60  0001 C CNN
-F 2 "antmicro-footprints:0402-cap" H 6800 3550 60  0001 L CNN
+F 2 "artix-dc-scm-footprints:0402-cap" H 6800 3550 60  0001 L CNN
 F 3 "" H 6600 3350 50  0001 C CNN
 F 4 "Walsin" H 6800 3750 60  0001 L CNN "Manufacturer"
@@
 $EndComp
 $Comp
-L antmicroCapacitors0402:C_100n_0402 C30
+L artix-dc-scm:C_100n_0402 C30
 U 1 1 5FD279FF
 P 6875 3450
 F 0 "C30" V 6617 3450 60  0000 C CNN
 F 1 "C_100n_0402" H 6875 3300 60  0001 C CNN
-F 2 "antmicro-footprints:0402-cap" H 7075 3650 60  0001 L CNN
+F 2 "artix-dc-scm-footprints:0402-cap" H 7075 3650 60  0001 L CNN
 F 3 "" H 6875 3450 50  0001 C CNN
 F 4 "Walsin" H 7075 3850 60  0001 L CNN "Manufacturer"
@@
 	3675 2750 4050 2750
 $Comp
-L antmicroResistors0402:R_10k_0402 R17
+L artix-dc-scm:R_10k_0402 R17
 U 1 1 5FD6D5E7
 P 3825 2125
 F 0 "R17" V 3780 2195 60  0000 L CNN
 F 1 "R_10k_0402" H 3825 1975 60  0001 C CNN
-F 2 "antmicro-footprints:0402-res" H 4025 2325 60  0001 L CNN
+F 2 "artix-dc-scm-footprints:0402-res" H 4025 2325 60  0001 L CNN
 F 3 "" H 3825 2125 50  0001 C CNN
 F 4 "VISHAY" H 4025 2525 60  0001 L CNN "Manufacturer"
@@
 $EndComp
 $Comp
-L antmicroResistors0402:R_10k_0402 R19
+L artix-dc-scm:R_10k_0402 R19
 U 1 1 5FD6DA61
 P 4050 2125
 F 0 "R19" V 4005 2195 60  0000 L CNN
 F 1 "R_10k_0402" H 4050 1975 60  0001 C CNN
-F 2 "antmicro-footprints:0402-res" H 4250 2325 60  0001 L CNN
+F 2 "artix-dc-scm-footprints:0402-res" H 4250 2325 60  0001 L CNN
 F 3 "" H 4050 2125 50  0001 C CNN
 F 4 "VISHAY" H 4250 2525 60  0001 L CNN "Manufacturer"
@@
 $EndComp
 $Comp
-L antmicroResistors0402:R_10k_0402 R20
+L artix-dc-scm:R_10k_0402 R20
 U 1 1 5FD7820E
 P 4275 2125
 F 0 "R20" V 4230 2195 60  0000 L CNN
 F 1 "R_10k_0402" H 4275 1975 60  0001 C CNN
-F 2 "antmicro-footprints:0402-res" H 4475 2325 60  0001 L CNN
+F 2 "artix-dc-scm-footprints:0402-res" H 4475 2325 60  0001 L CNN
 F 3 "" H 4275 2125 50  0001 C CNN
 F 4 "VISHAY" H 4475 2525 60  0001 L CNN "Manufacturer"
@@
 	4275 1500 4275 1975
 $Comp
-L antmicroLEDIndicationDiscrete:KP-1608CGCK D1
+L artix-dc-scm:KP-1608CGCK D1
 U 1 1 5FD7D8E8
 P 4250 4750
 F 0 "D1" H 4200 5087 60  0000 C CNN
 F 1 "KP-1608CGCK" H 4200 4981 60  0000 C CNN
-F 2 "antmicro-footprints:LED_0603" H 4450 4950 60  0001 L CNN
+F 2 "artix-dc-scm-footprints:LED_0603" H 4450 4950 60  0001 L CNN
 F 3 "http://www.farnell.com/datasheets/2045956.pdf" H 4450 5050 60  0001 L CNN
 F 4 "KP-1608CGCK" H 4450 5250 60  0001 L CNN "MPN"
@@
 	4350 4750 4650 4750
 $Comp
-L antmicroResistors0402:R_330R_0402 R18
+L artix-dc-scm:R_330R_0402 R18
 U 1 1 5FD7EE61
 P 3850 4375
 F 0 "R18" V 3805 4445 60  0000 L CNN
 F 1 "R_330R_0402" H 3850 4225 60  0001 C CNN
-F 2 "antmicro-footprints:0402-res" H 4050 4575 60  0001 L CNN
+F 2 "artix-dc-scm-footprints:0402-res" H 4050 4575 60  0001 L CNN
 F 3 "" H 3850 4375 50  0001 C CNN
 F 4 "MULTICOMP" H 4050 4775 60  0001 L CNN "Manufacturer"
@@
 	4550 5350 4550 5675
 $Comp
-L power:GND #PWR010
+L artix-dc-scm:GND #PWR010
 U 1 1 5FDC4FA1
 P 4550 5675
@@
 $EndComp
 $Comp
-L power:GND #PWR011
+L artix-dc-scm:GND #PWR011
 U 1 1 5FDC53F7
 P 6325 5675
@@
 $EndComp
 $Comp
-L antmicroCapacitors0402:C_10u_0402 C31
+L artix-dc-scm:C_10u_0402 C31
 U 1 1 5FDCA87A
 P 4850 6750
 F 0 "C31" H 4965 6795 60  0000 L CNN
 F 1 "C_10u_0402" H 4850 6600 60  0001 C CNN
-F 2 "antmicro-footprints:0402-cap" H 5050 6950 60  0001 L CNN
+F 2 "artix-dc-scm-footprints:0402-cap" H 5050 6950 60  0001 L CNN
 F 3 "" H 4850 6750 50  0001 C CNN
 F 4 "MURATA" H 5050 7150 60  0001 L CNN "Manufacturer"
@@
 $EndComp
 $Comp
-L antmicroCapacitors0402:C_10u_0402 C32
+L artix-dc-scm:C_10u_0402 C32
 U 1 1 5FDCB4B9
 P 5200 6750
 F 0 "C32" H 5315 6795 60  0000 L CNN
 F 1 "C_10u_0402" H 5200 6600 60  0001 C CNN
-F 2 "antmicro-footprints:0402-cap" H 5400 6950 60  0001 L CNN
+F 2 "artix-dc-scm-footprints:0402-cap" H 5400 6950 60  0001 L CNN
 F 3 "" H 5200 6750 50  0001 C CNN
 F 4 "MURATA" H 5400 7150 60  0001 L CNN "Manufacturer"
@@
 $EndComp
 $Comp
-L antmicroCapacitors0402:C_10u_0402 C33
+L artix-dc-scm:C_10u_0402 C33
 U 1 1 5FDCB85E
 P 5550 6750
 F 0 "C33" H 5665 6795 60  0000 L CNN
 F 1 "C_10u_0402" H 5550 6600 60  0001 C CNN
-F 2 "antmicro-footprints:0402-cap" H 5750 6950 60  0001 L CNN
+F 2 "artix-dc-scm-footprints:0402-cap" H 5750 6950 60  0001 L CNN
 F 3 "" H 5550 6750 50  0001 C CNN
 F 4 "MURATA" H 5750 7150 60  0001 L CNN "Manufacturer"
@@
 $EndComp
 $Comp
-L antmicroCapacitors0402:C_10u_0402 C34
+L artix-dc-scm:C_10u_0402 C34
 U 1 1 5FDCBB8F
 P 5900 6750
 F 0 "C34" H 6015 6795 60  0000 L CNN
 F 1 "C_10u_0402" H 5900 6600 60  0001 C CNN
-F 2 "antmicro-footprints:0402-cap" H 6100 6950 60  0001 L CNN
+F 2 "artix-dc-scm-footprints:0402-cap" H 6100 6950 60  0001 L CNN
 F 3 "" H 5900 6750 50  0001 C CNN
 F 4 "MURATA" H 6100 7150 60  0001 L CNN "Manufacturer"
@@
 $EndComp
 $Comp
-L power:GND #PWR012
+L artix-dc-scm:GND #PWR012
 U 1 1 5FDD1861
 P 4850 6900
@@
 $EndComp
 $Comp
-L power:GND #PWR013
+L artix-dc-scm:GND #PWR013
 U 1 1 5FDD1B5A
 P 5200 6900
@@
 $EndComp
 $Comp
-L power:GND #PWR014
+L artix-dc-scm:GND #PWR014
 U 1 1 5FDD1D85
 P 5550 6900
@@
 $EndComp
 $Comp
-L power:GND #PWR015
+L artix-dc-scm:GND #PWR015
 U 1 1 5FDD200B
 P 5900 6900
@@
 	6250 3950 6450 3950
 $Comp
-L antmicroCapacitors0402:C_100n_0402 C179
+L artix-dc-scm:C_100n_0402 C179
 U 1 1 5FFDF949
 P 6600 3950
 F 0 "C179" V 6342 3950 60  0000 C CNN
 F 1 "C_100n_0402" H 6600 3800 60  0001 C CNN
-F 2 "antmicro-footprints:0402-cap" H 6800 4150 60  0001 L CNN
+F 2 "artix-dc-scm-footprints:0402-cap" H 6800 4150 60  0001 L CNN
 F 3 "" H 6600 3950 50  0001 C CNN
 F 4 "Walsin" H 6800 4350 60  0001 L CNN "Manufacturer"
@@
 $EndComp
 $Comp
-L antmicroCapacitors0402:C_100n_0402 C181
+L artix-dc-scm:C_100n_0402 C181
 U 1 1 5FFDF952
 P 6875 4050
 F 0 "C181" V 6617 4050 60  0000 C CNN
 F 1 "C_100n_0402" H 6875 3900 60  0001 C CNN
-F 2 "antmicro-footprints:0402-cap" H 7075 4250 60  0001 L CNN
+F 2 "artix-dc-scm-footprints:0402-cap" H 7075 4250 60  0001 L CNN
 F 3 "" H 6875 4050 50  0001 C CNN
 F 4 "Walsin" H 7075 4450 60  0001 L CNN "Manufacturer"
@@
 	6775 4350 6250 4350
 $Comp
-L antmicroPciConnectors:1-2199230-6 J2
+L artix-dc-scm:1-2199230-6 J2
 U 1 1 5FD380A4
 P 5450 3900
 F 0 "J2" H 5450 6565 60  0000 C CNN
 F 1 "1-2199230-6" H 5300 2200 60  0001 C CNN
-F 2 "antmicro-footprints:1-2199230-6" H 5300 2200 60  0001 C CNN
+F 2 "artix-dc-scm-footprints:1-2199230-6" H 5300 2200 60  0001 C CNN
 F 3 "" H 5300 3900 60  0001 C CNN
 F 4 "TE" H 5450 6467 50  0000 C CNN "Manufacturer"
@@
 	6250 4550 6450 4550
 $Comp
-L antmicroCapacitors0402:C_100n_0402 C180
+L artix-dc-scm:C_100n_0402 C180
 U 1 1 60013CBE
 P 6600 4550
 F 0 "C180" V 6342 4550 60  0000 C CNN
 F 1 "C_100n_0402" H 6600 4400 60  0001 C CNN
-F 2 "antmicro-footprints:0402-cap" H 6800 4750 60  0001 L CNN
+F 2 "artix-dc-scm-footprints:0402-cap" H 6800 4750 60  0001 L CNN
 F 3 "" H 6600 4550 50  0001 C CNN
 F 4 "Walsin" H 6800 4950 60  0001 L CNN "Manufacturer"
@@
 $EndComp
 $Comp
-L antmicroCapacitors0402:C_100n_0402 C182
+L artix-dc-scm:C_100n_0402 C182
 U 1 1 60013CC7
 P 6875 4650
 F 0 "C182" V 6617 4650 60  0000 C CNN
 F 1 "C_100n_0402" H 6875 4500 60  0001 C CNN
-F 2 "antmicro-footprints:0402-cap" H 7075 4850 60  0001 L CNN
+F 2 "artix-dc-scm-footprints:0402-cap" H 7075 4850 60  0001 L CNN
 F 3 "" H 6875 4650 50  0001 C CNN
 F 4 "Walsin" H 7075 5050 60  0001 L CNN "Manufacturer"
