File: pcie-conn.sch (KiCad schematic (older format))
At the start: 22 parts, among them J2 1-2199230-6

Commit message: Update component libraries
Parts:
- C179, C180, C181, C182, C27, C28, C29, C30: symbol artix-dc-scm:C_100n_0402 -> artix-dc-scm:C_100n_0402-artix-dc-scm
- TP12, TP13, TP14: footprint antmicro-footprints:Testpoint_smd_1mm -> artix-dc-scm-footprints:Testpoint_smd_1mm
Changed lines of the file:
@@
 	6250 2750 6450 2750
 $Comp
-L artix-dc-scm:C_100n_0402 C27
+L artix-dc-scm:C_100n_0402-artix-dc-scm C27
 U 1 1 5FD1CF34
 P 6600 2750
@@
 $EndComp
 $Comp
-L artix-dc-scm:C_100n_0402 C29
+L artix-dc-scm:C_100n_0402-artix-dc-scm C29
 U 1 1 5FD1DAE4
 P 6875 2850
@@
 	6250 3350 6450 3350
 $Comp
-L artix-dc-scm:C_100n_0402 C28
+L artix-dc-scm:C_100n_0402-artix-dc-scm C28
 U 1 1 5FD279F6
 P 6600 3350
@@
 $EndComp
 $Comp
-L artix-dc-scm:C_100n_0402 C30
+L artix-dc-scm:C_100n_0402-artix-dc-scm C30
 U 1 1 5FD279FF
 P 6875 3450
@@
 	4550 5350 4550 5675
 $Comp
-L artix-dc-scm:GND #PWR010
+L artix-dc-scm:GND-artix-dc-scm #PWR010
 U 1 1 5FDC4FA1
 P 4550 5675
@@
 $EndComp
 $Comp
-L artix-dc-scm:GND #PWR011
+L artix-dc-scm:GND-artix-dc-scm #PWR011
 U 1 1 5FDC53F7
 P 6325 5675
@@
 $EndComp
 $Comp
-L artix-dc-scm:GND #PWR012
+L artix-dc-scm:GND-artix-dc-scm #PWR012
 U 1 1 5FDD1861
 P 4850 6900
@@
 $EndComp
 $Comp
-L artix-dc-scm:GND #PWR013
+L artix-dc-scm:GND-artix-dc-scm #PWR013
 U 1 1 5FDD1B5A
 P 5200 6900
@@
 $EndComp
 $Comp
-L artix-dc-scm:GND #PWR014
+L artix-dc-scm:GND-artix-dc-scm #PWR014
 U 1 1 5FDD1D85
 P 5550 6900
@@
 $EndComp
 $Comp
-L artix-dc-scm:GND #PWR015
+L artix-dc-scm:GND-artix-dc-scm #PWR015
 U 1 1 5FDD200B
 P 5900 6900
@@
 	6250 3950 6450 3950
 $Comp
-L artix-dc-scm:C_100n_0402 C179
+L artix-dc-scm:C_100n_0402-artix-dc-scm C179
 U 1 1 5FFDF949
 P 6600 3950
@@
 $EndComp
 $Comp
-L artix-dc-scm:C_100n_0402 C181
+L artix-dc-scm:C_100n_0402-artix-dc-scm C181
 U 1 1 5FFDF952
 P 6875 4050
@@
 	6250 4550 6450 4550
 $Comp
-L artix-dc-scm:C_100n_0402 C180
+L artix-dc-scm:C_100n_0402-artix-dc-scm C180
 U 1 1 60013CBE
 P 6600 4550
@@
 $EndComp
 $Comp
-L artix-dc-scm:C_100n_0402 C182
+L artix-dc-scm:C_100n_0402-artix-dc-scm C182
 U 1 1 60013CC7
 P 6875 4650
@@
 F 0 "TP12" V 3480 2597 50  0000 C CNN
 F 1 "TP_SMD1MM" H 3575 2450 50  0001 C CNN
-F 2 "antmicro-footprints:Testpoint_smd_1mm" H 3775 2750 60  0001 L CNN
+F 2 "artix-dc-scm-footprints:Testpoint_smd_1mm" H 3775 2750 60  0001 L CNN
 F 3 "" H 3775 2850 60  0001 L CNN
 	1    3575 2550
@@
 F 0 "TP13" V 3480 2697 50  0000 C CNN
 F 1 "TP_SMD1MM" H 3575 2550 50  0001 C CNN
-F 2 "antmicro-footprints:Testpoint_smd_1mm" H 3775 2850 60  0001 L CNN
+F 2 "artix-dc-scm-footprints:Testpoint_smd_1mm" H 3775 2850 60  0001 L CNN
 F 3 "" H 3775 2950 60  0001 L CNN
 	1    3575 2650
@@
 F 0 "TP14" H 3875 2897 50  0000 L CNN
 F 1 "TP_SMD1MM" H 3825 2750 50  0001 C CNN
-F 2 "antmicro-footprints:Testpoint_smd_1mm" H 4025 3050 60  0001 L CNN
+F 2 "artix-dc-scm-footprints:Testpoint_smd_1mm" H 4025 3050 60  0001 L CNN
 F 3 "" H 4025 3150 60  0001 L CNN
 	1    3825 2850
