File: pcie-conn.sch (KiCad schematic (older format))
At the start: 22 parts, among them J2 1-2199230-6

Commit message: Fixed libs
Parts:
- C179, C180, C181, C182, C27, C28, C29, C30: footprint _autosave-artix-dc-scm-footprints:0402-cap -> artix-dc-scm-footprints:0402-cap; symbol _autosave-artix-dc-scm:C_100n_0402-artix-dc-scm -> artix-dc-scm:C_100n_0402-artix-dc-scm
- C31, C32, C33, C34: footprint _autosave-artix-dc-scm-footprints:0402-cap -> artix-dc-scm-footprints:0402-cap; symbol _autosave-artix-dc-scm:C_10u_0402 -> artix-dc-scm:C_10u_0402
- D1: footprint _autosave-artix-dc-scm-footprints:LED_0603 -> artix-dc-scm-footprints:LED_0603; symbol _autosave-artix-dc-scm:KP-1608CGCK -> artix-dc-scm:KP-1608CGCK
- J2: footprint _autosave-artix-dc-scm-footprints:1-2199230-6 -> artix-dc-scm-footprints:1-2199230-6; symbol _autosave-artix-dc-scm:1-2199230-6 -> artix-dc-scm:1-2199230-6
- R17, R19, R20: footprint _autosave-artix-dc-scm-footprints:0402-res -> artix-dc-scm-footprints:0402-res; symbol _autosave-artix-dc-scm:R_10k_0402 -> artix-dc-scm:R_10k_0402
- R18: footprint _autosave-artix-dc-scm-footprints:0402-res -> artix-dc-scm-footprints:0402-res; symbol _autosave-artix-dc-scm:R_330R_0402 -> artix-dc-scm:R_330R_0402
- SP1: footprint _autosave-artix-dc-scm-footprints:9774025151 -> artix-dc-scm-footprints:9774025151; symbol _autosave-artix-dc-scm:9774025151 -> artix-dc-scm:9774025151
- TP12, TP13, TP14: footprint _autosave-artix-dc-scm-footprints:Testpoint_smd_1mm -> artix-dc-scm-footprints:Testpoint_smd_1mm; symbol _autosave-artix-dc-scm:TP_SMD1MM -> artix-dc-scm:TP_SMD1MM
